File: hardware/eagle/p8x-backplane.brd (EAGLE design)
At the start: 248.9 x 109.2 mm, 30 parts, among them J1 SLOT1, J10 SLOT10, J11 PWR-5V, J2 SLOT2, J3 SLOT3, J4 SLOT4, J5 SLOT5, J6 SLOT6, J7 SLOT7, J8 SLOT8, J9 SLOT9

Commit message: redo all files
Connections:
- net SPARE0 renamed FC
- net SPARE1 renamed FZ
- net SPARE2 renamed FN
- net SPARE3 renamed FV
- new net SPARE10: J1.B29, J10.B29, J2.B29, J3.B29, J4.B29, J5.B29, J6.B29, J7.B29, J8.B29, J9.B29
- new net SPARE11: J1.B30, J10.B30, J2.B30, J3.B30, J4.B30, J5.B30, J6.B30, J7.B30, J8.B30, J9.B30
- new net SPARE8: J1.B27, J10.B27, J2.B27, J3.B27, J4.B27, J5.B27, J6.B27, J7.B27, J8.B27, J9.B27
- new net SPARE9: J1.B28, J10.B28, J2.B28, J3.B28, J4.B28, J5.B28, J6.B28, J7.B28, J8.B28, J9.B28
- net GND: no longer J1.B27, J1.B28, J1.B29, J1.B30, J10.B27, J10.B28, J10.B29, J10.B30, J2.B27, J2.B28, J2.B29, J2.B30, J3.B27, J3.B28, J3.B29, J3.B30, J4.B27, J4.B28, J4.B29, J4.B30, J5.B27, J5.B28, J5.B29, J5.B30, J6.B27, J6.B28, J6.B29, J6.B30, J7.B27, J7.B28, J7.B29, J7.B30, J8.B27, J8.B28, J8.B29, J8.B30, J9.B27, J9.B28, J9.B29, J9.B30
Routing:
- net SPARE9: track 0.00 -> 241.3 mm
- net SPARE8: track 0.00 -> 241.3 mm
- net SPARE11: track 0.00 -> 241.3 mm
- net SPARE10: track 0.00 -> 241.3 mm
