File: hardware/backplane/p8x-backplane.sch (EAGLE design)
At the start: 30 parts, among them J1 SLOT1, J10 SLOT10, J11 PWR-5V, J2 SLOT2, J3 SLOT3, J4 SLOT4, J5 SLOT5, J6 SLOT6, J7 SLOT7, J8 SLOT8, J9 SLOT9

Commit message: hw(rev C3): allocate backplane lines for the rev-B control signals
Phase 2, step 1 (bus contract). busnet() reassigns spares to the rev-B
microcode-word signals: C27-C30 = PSEL2/LDZN/SHCIN/SETC, B27 = CLRC
(were SPARE4-8); SPARE9-11 remain on B28-B30. The backplane buses them
to all 10 slots automatically; cards consume them in later steps
(control card drives them; reg-bank uses PSEL2; ALU uses the rest).

Updated bus-definition.md (pinout, spare notes, full rev-B microcode
word layout, revision history) and gen_bus_pdf.py (matching busnet copy
+ signal descriptions); regenerated the backplane and bus PDF. Also
gitignore stray root u*.bin from running a generator in the repo root.

Co-Authored-By: Claude Opus 4.8 <noreply@anthropic.com>
Connections:
- net SPARE4 renamed PSEL2
- net SPARE5 renamed LDZN
- net SPARE6 renamed SHCIN
- net SPARE7 renamed SETC
- net SPARE8 renamed CLRC
Changed lines of the file:
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@@
 <label x="515.62" y="-723.39" size="1.778" layer="95"/></segment>
 </net>
-<net name="SPARE8" class="0">
+<net name="CLRC" class="0">
 <segment><pinref part="J1" gate="G$1" pin="B27"/>
 <wire x1="17.78" y1="-109.22" x2="12.70" y2="-109.22" width="0.1524" layer="91"/>
@@
 <label x="464.82" y="-306.83" size="1.778" layer="95"/></segment>
 </net>
-<net name="SPARE4" class="0">
+<net name="PSEL2" class="0">
 <segment><pinref part="J1" gate="G$1" pin="C27"/>
 <wire x1="53.34" y1="-27.94" x2="58.42" y2="-27.94" width="0.1524" layer="91"/>
@@
 <label x="464.82" y="-309.37" size="1.778" layer="95"/></segment>
 </net>
-<net name="SPARE5" class="0">
+<net name="LDZN" class="0">
 <segment><pinref part="J1" gate="G$1" pin="C28"/>
 <wire x1="53.34" y1="-30.48" x2="58.42" y2="-30.48" width="0.1524" layer="91"/>
@@
 <label x="464.82" y="-311.91" size="1.778" layer="95"/></segment>
 </net>
-<net name="SPARE6" class="0">
+<net name="SHCIN" class="0">
 <segment><pinref part="J1" gate="G$1" pin="C29"/>
 <wire x1="53.34" y1="-33.02" x2="58.42" y2="-33.02" width="0.1524" layer="91"/>
@@
 <label x="464.82" y="-314.45" size="1.778" layer="95"/></segment>
 </net>
-<net name="SPARE7" class="0">
+<net name="SETC" class="0">
 <segment><pinref part="J1" gate="G$1" pin="C30"/>
 <wire x1="53.34" y1="-35.56" x2="58.42" y2="-35.56" width="0.1524" layer="91"/>

Commit message: feat: 2nd ALU-input mux (rev C) — B-side operand can select T
Add a 2:1 mux on the ALU B-operand path so the second ALU operand can be
the T register instead of B, controlled by a new microcode-word bit.

- microcode (genucode.py): BSEL = word bit 31 (was the lone spare); new
  opcodes ADDT/SUBT/ANDT/ORT/XORT/CMPT (0x80-0x85) run the ALU with T as
  the B operand (B preserved); LDT #imm / LDT a (0x86/0x87) expose T, which
  was microcode-scratch-only and had no programmer-visible load.
- emulator (p8xemu.c): decode bit 31; ALU B operand = bsel ? T : B.
- hardware (gen_eagle.py): ALU card U32/U33 (74157 x2) mux BQ vs TQ -> 74181 B;
  BSEL latched in control-card pipe U17.Q8, carried on backplane B28 (was
  SPARE9). All 7 boards regenerate with 0 validation errors.
- bus map kept consistent across both generators (gen_eagle.py, gen_bus_pdf.py),
  the backplane render, and the hardware docs (bus-definition is authoritative).
- tests: new ISA coverage for the T-operand ops (sentinel wrong-operand bait);
  all 6 suites pass.
- docs: programmer's guide regenerated; BACKLOG updated (mux -> DONE; added a
  post-bringup idea to optimize monitor/OS/BASIC hot paths with the T ops).

Backward-compatible: no existing opcode changed; BSEL defaults 0 (= B register),
so existing monitor/OS/BASIC binaries are byte-identical.

Co-Authored-By: Claude Opus 4.8 <noreply@anthropic.com>
Connections:
- net SPARE9 renamed BSEL
Changed lines of the file:
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@@
 <label x="419.10" y="-390.65" size="1.778" layer="95"/></segment>
 </net>
-<net name="SPARE9" class="0">
+<net name="BSEL" class="0">
 <segment><pinref part="J1" gate="G$1" pin="B28"/>
 <wire x1="17.78" y1="-111.76" x2="12.70" y2="-111.76" width="0.1524" layer="91"/>

Commit message: feat(hw): provision IRQ controller footprints (DNP) + reserve IRQ bus line
Per the chosen conservative path: add the interrupt-controller footprints and
the IRQ bus line so the controller can be built post-fab without a respin, but
WITHOUT the bus-critical logic that could brick an unvalidated board.

- Control card: U20 (74244 forcing buffer) + U21 (7474 IE/pending FF) placed as
  DNP. Safe connections wired: U20 inputs = $08 pattern, U20 !G tied high
  (outputs forced high-Z), IRQ line -> U21. Left UNWIRED (bus-critical, design
  with DRC first): U20 outputs onto the data bus, the enable/service sequencer,
  the EI/DI/RTI opcode decode, and the cross-card memory -RD suppression.
- Backplane: B29 = IRQ (was SPARE10), reserved; SPARE11 remains on B30.
- Bus map kept consistent across both generators + the backplane render + the
  three hardware docs (bus-definition is authoritative). Programmer's guide and
  BACKLOG updated.

All 7 boards regenerate with 0 validation errors; all 6 test suites pass.

Co-Authored-By: Claude Opus 4.8 <noreply@anthropic.com>
Connections:
- net SPARE10 renamed IRQ
Changed lines of the file:
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@@
 <label x="419.10" y="-393.19" size="1.778" layer="95"/></segment>
 </net>
-<net name="SPARE10" class="0">
+<net name="IRQ" class="0">
 <segment><pinref part="J1" gate="G$1" pin="B29"/>
 <wire x1="17.78" y1="-114.30" x2="12.70" y2="-114.30" width="0.1524" layer="91"/>

Commit message: feat(backplane): row-B even pins become spare bus lines (SPARE12-23)
Row B was a solid ground guard (B3-26 all GND). Per request, B3-26 now ALTERNATE:
odd pins stay GND (still a guard between most signal pairs), and the 12 even pins
(B4,B6,..,B26) become spare bus lines SPARE12-SPARE23, routed slot-to-slot — so
new signals can be added later without re-spinning the backplane. B27-30
(CLRC/BSEL/IRQ/SPARE11) unchanged.

- busnet() updated in all three copies (gen_eagle, gen_bus_pdf, gen_bus_card)
- backplane .brd routes the 12 new spares (mirrors the B27-30 routing); odd-pin
  grounds remain on the GND pour
- every card regenerated: their connectors no longer tie the even B pins to GND
  (those are spare lines now) — they simply don't connect the spares
- all 8 boards validate (0 errors); schematic + bus PDFs regenerated
- docs updated: bus-definition (pin map + notes), backplane theory + design notes
- net signal-integrity trade noted: a solid guard shields slightly better; the
  alternation was chosen deliberately for expansion room

Co-Authored-By: Claude Opus 4.8 <noreply@anthropic.com>
Connections:
- new net SPARE12: J1.B4, J10.B4, J2.B4, J3.B4, J4.B4, J5.B4, J6.B4, J7.B4, J8.B4, J9.B4
- new net SPARE13: J1.B6, J10.B6, J2.B6, J3.B6, J4.B6, J5.B6, J6.B6, J7.B6, J8.B6, J9.B6
- new net SPARE14: J1.B8, J10.B8, J2.B8, J3.B8, J4.B8, J5.B8, J6.B8, J7.B8, J8.B8, J9.B8
- new net SPARE15: J1.B10, J10.B10, J2.B10, J3.B10, J4.B10, J5.B10, J6.B10, J7.B10, J8.B10, J9.B10
- new net SPARE16: J1.B12, J10.B12, J2.B12, J3.B12, J4.B12, J5.B12, J6.B12, J7.B12, J8.B12, J9.B12
- new net SPARE17: J1.B14, J10.B14, J2.B14, J3.B14, J4.B14, J5.B14, J6.B14, J7.B14, J8.B14, J9.B14
- new net SPARE18: J1.B16, J10.B16, J2.B16, J3.B16, J4.B16, J5.B16, J6.B16, J7.B16, J8.B16, J9.B16
- new net SPARE19: J1.B18, J10.B18, J2.B18, J3.B18, J4.B18, J5.B18, J6.B18, J7.B18, J8.B18, J9.B18
- new net SPARE20: J1.B20, J10.B20, J2.B20, J3.B20, J4.B20, J5.B20, J6.B20, J7.B20, J8.B20, J9.B20
- new net SPARE21: J1.B22, J10.B22, J2.B22, J3.B22, J4.B22, J5.B22, J6.B22, J7.B22, J8.B22, J9.B22
- new net SPARE22: J1.B24, J10.B24, J2.B24, J3.B24, J4.B24, J5.B24, J6.B24, J7.B24, J8.B24, J9.B24
- new net SPARE23: J1.B26, J10.B26, J2.B26, J3.B26, J4.B26, J5.B26, J6.B26, J7.B26, J8.B26, J9.B26
- net GND: no longer J1.B10, J1.B12, J1.B14, J1.B16, J1.B18, J1.B20, J1.B22, J1.B24, J1.B26, J1.B4, J1.B6, J1.B8, J10.B10, J10.B12, J10.B14, J10.B16, J10.B18, J10.B20, J10.B22, J10.B24, J10.B26, J10.B4, J10.B6, J10.B8, J2.B10, J2.B12, J2.B14, J2.B16, J2.B18, J2.B20, J2.B22, J2.B24, J2.B26, J2.B4, J2.B6, J2.B8, J3.B10, J3.B12, J3.B14, J3.B16, J3.B18, J3.B20, J3.B22, J3.B24, J3.B26, J3.B4, J3.B6, J3.B8, J4.B10, J4.B12, J4.B14, J4.B16, J4.B18, J4.B20, J4.B22, J4.B24, J4.B26, J4.B4, J4.B6, J4.B8, J5.B10, J5.B12, J5.B14, J5.B16, J5.B18, J5.B20, J5.B22, J5.B24, J5.B26, J5.B4, J5.B6, J5.B8, J6.B10, J6.B12, J6.B14, J6.B16, J6.B18, J6.B20, J6.B22, J6.B24, J6.B26, J6.B4, J6.B6, J6.B8, J7.B10, J7.B12, J7.B14, J7.B16, J7.B18, J7.B20, J7.B22, J7.B24, J7.B26, J7.B4, J7.B6, J7.B8, J8.B10, J8.B12, J8.B14, J8.B16, J8.B18, J8.B20, J8.B22, J8.B24, J8.B26, J8.B4, J8.B6, J8.B8, J9.B10, J9.B12, J9.B14, J9.B16, J9.B18, J9.B20, J9.B22, J9.B24, J9.B26, J9.B4, J9.B6, J9.B8
