File: hardware/led-card/p8x-led-card.brd (EAGLE design)
At the start: 160 x 100 mm, 19 parts, among them J1 FABC96R, U1 IO PAGE, U2 ADDR DEC, U3 DLD DEC, U4 74HCT32, U5 74HCT14, U6 LED LATCH

Commit message: feat(backplane): row-B even pins become spare bus lines (SPARE12-23)
Row B was a solid ground guard (B3-26 all GND). Per request, B3-26 now ALTERNATE:
odd pins stay GND (still a guard between most signal pairs), and the 12 even pins
(B4,B6,..,B26) become spare bus lines SPARE12-SPARE23, routed slot-to-slot — so
new signals can be added later without re-spinning the backplane. B27-30
(CLRC/BSEL/IRQ/SPARE11) unchanged.

- busnet() updated in all three copies (gen_eagle, gen_bus_pdf, gen_bus_card)
- backplane .brd routes the 12 new spares (mirrors the B27-30 routing); odd-pin
  grounds remain on the GND pour
- every card regenerated: their connectors no longer tie the even B pins to GND
  (those are spare lines now) — they simply don't connect the spares
- all 8 boards validate (0 errors); schematic + bus PDFs regenerated
- docs updated: bus-definition (pin map + notes), backplane theory + design notes
- net signal-integrity trade noted: a solid guard shields slightly better; the
  alternation was chosen deliberately for expansion room

Co-Authored-By: Claude Opus 4.8 <noreply@anthropic.com>
Connections:
- net GND: no longer J1.B10, J1.B12, J1.B14, J1.B16, J1.B18, J1.B20, J1.B22, J1.B24, J1.B26, J1.B4, J1.B6, J1.B8
Changed lines of the file:
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@@
 <contactref element="J1" pad="A32"/>
 <contactref element="J1" pad="B3"/>
-<contactref element="J1" pad="B4"/>
 <contactref element="J1" pad="B5"/>
-<contactref element="J1" pad="B6"/>
 <contactref element="J1" pad="B7"/>
-<contactref element="J1" pad="B8"/>
 <contactref element="J1" pad="B9"/>
-<contactref element="J1" pad="B10"/>
 <contactref element="J1" pad="B11"/>
-<contactref element="J1" pad="B12"/>
 <contactref element="J1" pad="B13"/>
-<contactref element="J1" pad="B14"/>
 <contactref element="J1" pad="B15"/>
-<contactref element="J1" pad="B16"/>
 <contactref element="J1" pad="B17"/>
-<contactref element="J1" pad="B18"/>
 <contactref element="J1" pad="B19"/>
-<contactref element="J1" pad="B20"/>
 <contactref element="J1" pad="B21"/>
-<contactref element="J1" pad="B22"/>
 <contactref element="J1" pad="B23"/>
-<contactref element="J1" pad="B24"/>
 <contactref element="J1" pad="B25"/>
-<contactref element="J1" pad="B26"/>
 <contactref element="J1" pad="B31"/>
 <contactref element="J1" pad="B32"/>

Commit message: feat(generators): faithful Eagle/Fusion output (values, layers, smashed parts)
Make the generated .sch/.brd match how Eagle itself writes files, so Fusion
displays everything correctly (was mis-mapping names/values to scratch layers):

- devicesets get uservalue="yes" so the `value` field is honored at all (it was
  silently ignored before — no card's value ever displayed)
- emit the COMPLETE standard Eagle layer table (62 layers) in every drawing, so
  Fusion has nothing to remap on import
- board elements are now smashed="yes" with explicit NAME (tNames/25) and VALUE
  (tValues/27) attributes — refdes + part number show reliably
- add std <attributes>/<variantdefs> board sections + board-package >VALUE silk
- schematic: `value` holds the orderable part number (>VALUE + BOM); the logical
  function is placed as text near each chip via a new card() `labels` arg
- write_brd gains outline_only and unplaced modes (parts off-board + ratsnest);
  card() exposes brd_outline_only / brd_unplaced

Proven on the LED card (part numbers + function labels + an unplaced 4-layer
board). The other cards get the structural fixes now; rolling the part-number/
labels convention across them is the next step. All 8 boards validate (0 errors).

Co-Authored-By: Claude Opus 4.8 <noreply@anthropic.com>
Parts:
- LA1: value OUT LEDS -> 8-LED BAR
- LED3: value PWR-GRN -> GRN
- LED4: value WR-YEL -> YEL
- RL1: value 8X330R -> 8x330R
- U1: value IO PAGE -> 74HCT30
- U2: value ADDR DEC -> 74HCT138
- U3: value DLD DEC -> 74HCT138
- U6: value LED LATCH -> 74HCT374
- moved CD4 185.4 mm to (263.9, 95.1)
- moved RL1 185.4 mm to (300.6, 97.7)
- moved U5 185.4 mm to (268.2, 95.2)
- moved CD6 185.4 mm to (296.3, 95.1)
- moved J1 185.4 mm to (190.8, 87.0)
- moved LA1 185.4 mm to (304.8, 95.2)
- moved LED4 185.4 mm to (217.7, 52.8)
- moved R4 185.4 mm to (203.3, 52.9)
- moved RP1 185.4 mm to (316.6, 95.2)
- moved U1 185.4 mm to (203.3, 95.2)
- moved U2 185.4 mm to (219.5, 95.2)
- moved U3 185.4 mm to (235.7, 95.2)
- moved CD1 185.4 mm to (215.2, 95.1)
- moved CD2 185.4 mm to (231.4, 95.1)
- moved CD3 185.4 mm to (247.6, 95.1)
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Routing:
- removed copper zone on layer 2, net GND
- removed copper zone on layer 15, net VCC

Commit message: feat(hardware): use con-vg DIN 41612 footprints (MABC96R card / FABC96S backplane)
Replace the hand-rolled DIN96/DIN96C connector packages with the real Eagle
con-vg DIN 41612 footprints (geometry baked into the generator so it stays
self-contained): card edge = MABC96R (male right-angle), backplane = FABC96S
(female vertical) — both A/B/C @ 2.54mm, drill 0.9144, two M2.5 mounting holes
at y=+/-45. Card value -> MABC96R; pin->pad names unchanged (A1..C32) so the
netlist is intact.

con-vg centres the pad field on the element origin, so the backplane (hand-
placed/routed) was re-derived: slots dropped to y=54.6 to centre the pin field
on the 109mm board (pads now on-board), bus traces re-routed to the new A/B/C
columns (element at sx(i)-2.54). Cards auto-adapt via fp_box. All 8 boards
validate (0 errors).

Known: 3 placement-overlap WARNINGS on the backplane (power-LED resistor; CT2/RT1
clock terminators, both DNP) where the taller connector crowds the top/bottom
strips — to clear during the Fusion placement pass.

Co-Authored-By: Claude Opus 4.8 <noreply@anthropic.com>
Parts:
- J1: value FABC96R -> MABC96R; device p8x:DIN96C -> p8x:MABC96R
- moved J1 37.5 mm to (193.3, 49.6)

Commit message: feat(hardware): 100nF bypass caps to 0.1" lead pitch on all boards
The 100nF ceramic-disc decoupling/bypass caps used the shared C_DISC footprint
at 0.2" (5.08mm) lead spacing. The parts being sourced are 0.1" (2.54mm) pitch,
so retarget just those caps:

- Add a C_DISC1 footprint (pad 2 at y=-2.54) and a CAP1 device that reuses the
  CAP schematic symbol art but points at C_DISC1.
- Route the 100nF parts to CAP1: per-IC decoupling (CDn), the placement-flow
  copies, and the backplane per-slot caps C1-C10.
- Leave C_DISC (0.2") for the parts that still use it: the 1uF caps, the 150pF
  clock terminators (CT1/CT2), and the XTAL32 placeholder.

Regenerated all 8 boards (.sch/.brd/-full.brd) and the schematic PDFs; the
narrower pad field also relieves the backplane connector clearance. Validation:
0 errors on all boards.

Co-Authored-By: Claude Opus 4.8 <noreply@anthropic.com>
Parts:
- CD1, CD2, CD3, CD4, CD5, CD6: device p8x:C_DISC -> p8x:C_DISC1
Changed lines of the file:
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@@
 <attribute name="VALUE" x="203.27" y="92.66" size="1.778" layer="27" ratio="10"/>
 </element>
-<element name="CD1" library="p8x" package="C_DISC" value="100N" x="215.19" y="95.10" smashed="yes">
+<element name="CD1" library="p8x" package="C_DISC1" value="100N" x="215.19" y="95.10" smashed="yes">
 <attribute name="NAME" x="215.19" y="97.64" size="1.778" layer="25" ratio="10"/>
 <attribute name="VALUE" x="215.19" y="92.56" size="1.778" layer="27" ratio="10"/>
@@
 <attribute name="VALUE" x="219.49" y="92.66" size="1.778" layer="27" ratio="10"/>
 </element>
-<element name="CD2" library="p8x" package="C_DISC" value="100N" x="231.41" y="95.10" smashed="yes">
+<element name="CD2" library="p8x" package="C_DISC1" value="100N" x="231.41" y="95.10" smashed="yes">
 <attribute name="NAME" x="231.41" y="97.64" size="1.778" layer="25" ratio="10"/>
 <attribute name="VALUE" x="231.41" y="92.56" size="1.778" layer="27" ratio="10"/>
@@
 <attribute name="VALUE" x="235.71" y="92.66" size="1.778" layer="27" ratio="10"/>
 </element>
-<element name="CD3" library="p8x" package="C_DISC" value="100N" x="247.63" y="95.10" smashed="yes">
+<element name="CD3" library="p8x" package="C_DISC1" value="100N" x="247.63" y="95.10" smashed="yes">
 <attribute name="NAME" x="247.63" y="97.64" size="1.778" layer="25" ratio="10"/>
 <attribute name="VALUE" x="247.63" y="92.56" size="1.778" layer="27" ratio="10"/>
@@
 <attribute name="VALUE" x="251.93" y="92.66" size="1.778" layer="27" ratio="10"/>
 </element>
-<element name="CD4" library="p8x" package="C_DISC" value="100N" x="263.85" y="95.10" smashed="yes">
+<element name="CD4" library="p8x" package="C_DISC1" value="100N" x="263.85" y="95.10" smashed="yes">
 <attribute name="NAME" x="263.85" y="97.64" size="1.778" layer="25" ratio="10"/>
 <attribute name="VALUE" x="263.85" y="92.56" size="1.778" layer="27" ratio="10"/>
@@
 <attribute name="VALUE" x="268.15" y="92.66" size="1.778" layer="27" ratio="10"/>
 </element>
-<element name="CD5" library="p8x" package="C_DISC" value="100N" x="280.07" y="95.10" smashed="yes">
+<element name="CD5" library="p8x" package="C_DISC1" value="100N" x="280.07" y="95.10" smashed="yes">
 <attribute name="NAME" x="280.07" y="97.64" size="1.778" layer="25" ratio="10"/>
 <attribute name="VALUE" x="280.07" y="92.56" size="1.778" layer="27" ratio="10"/>
@@
 <attribute name="VALUE" x="284.37" y="92.66" size="1.778" layer="27" ratio="10"/>
 </element>
-<element name="CD6" library="p8x" package="C_DISC" value="100N" x="296.29" y="95.10" smashed="yes">
+<element name="CD6" library="p8x" package="C_DISC1" value="100N" x="296.29" y="95.10" smashed="yes">
 <attribute name="NAME" x="296.29" y="97.64" size="1.778" layer="25" ratio="10"/>
 <attribute name="VALUE" x="296.29" y="92.56" size="1.778" layer="27" ratio="10"/>
