File: hardware/xor-trial/kicad/xor_trial.kicad_pcb (KiCad board)
At the start: 2 copper layers, 62 x 44 mm, 9 parts, among them J1 +5V/GND, SW1 PUSH, SW2 PUSH, U1 74HC86

Commit message: feat(xor-trial): add KiCad schematic (ERC-clean) + power-header +/- silk
Add gen_sch.py, a second generator for the XOR trial board that emits the
schematic (xor_trial.kicad_sch, + PDF) to match gen_xor.py's board. It hand-codes
the same netlist and passes `kicad-cli sch erc` clean (0 violations): one 74HC86
(gate 1 used, spare gates grounded with no-connect outputs), two buttons with 10k
pull-downs, an LED through 330R on the output, a 100nF decoupler, and a J1 power
entry with +5V/GND power symbols and a PWR_FLAG per rail.

gen_sch.py lifts full symbol defs out of the installed .kicad_sym libs with
kiutils (no geometry hand-copied) but emits the modern KiCad-8 (20231120) file
itself: kiutils only writes the KiCad-6 format, which KiCad 10's net/ERC engine
does not read back (netlist export returns zero components, so ERC "passes" on an
empty sheet -- a false clean). The XOR part is placed as the concrete 74xx:74LS86
base symbol valued "74HC86", because a hand-flattened copy of the derived 74HC86
trips ERC's lib_symbol_mismatch check. Everything sits on the 1.27 mm grid so no
pin lands off-grid.

Also add + / - silkscreen labels next to the power header on the board
(gen_xor.py), and regenerate the board + gerber zip. Board still DRC-clean
(0 violations, 0 unconnected). READMEs updated.

Co-Authored-By: Claude Opus 4.8 <noreply@anthropic.com>
Other:
- board text added: "+"
- board text added: "-"
