File: hardware/led-card/kicad/p8x-led-card.kicad_pcb (KiCad board)
At the start: 4 copper layers, 200 x 100 mm, 19 parts, among them J1 MABC96R, U1 74HCT30, U2 74HCT138, U3 74HCT138, U4 74HCT32, U5 74HCT14, U6 74HCT374

Commit message: feat(kicad): re-route led/cf/control/io/alu at uniform 280x140mm
All cards rebuilt at the uniform 280x140 size with the unified courtyard-spaced
placement (0 hard DRC violations) and re-routed with Freerouting.

Co-Authored-By: Claude Opus 4.8 <noreply@anthropic.com>
Parts:
- moved RL1 156.5 mm to (212.7, 9.82)
- moved LA1 154.3 mm to (186.5, 16.7)
- moved LED4 75.9 mm to (267.7, 11.3), turned to 0 degrees
- moved R4 69.0 mm to (238.0, 9.54)
- moved LED3 62.9 mm to (256.2, 11.3), turned to 0 degrees
- moved RP1 49.8 mm to (220.6, 9.54)
- moved J1 20.0 mm to (6.54, 109.4)
- moved C6 10.3 mm to (164.5, 10.6)
- moved U6 10.3 mm to (155.6, 22.7)
- moved U5 8.14 mm to (132.2, 22.7)
- moved C5 8.14 mm to (137.3, 10.6)
- moved C4 6.00 mm to (113.9, 10.6)
- moved U4 6.00 mm to (108.8, 22.7)
- moved C3 3.87 mm to (89.3, 10.6)
- moved U3 3.87 mm to (82.9, 22.7)
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Routing:
- net LP4: track 143.6 -> 46.2 mm, vias 1 -> 0
- net LP3: track 117.9 -> 37.8 mm
- net WRSEL: track 89.7 -> 160.2 mm
- net LP5: track 118.9 -> 52.8 mm
- net LP2: track 108.1 -> 45.6 mm
- net LP6: track 118.1 -> 57.4 mm
- net LP1: track 103.5 -> 50.2 mm
- net LP7: track 112.0 -> 68.4 mm
- net A9: track 49.9 -> 86.7 mm
- net LP0: track 93.8 -> 60.0 mm
- net A1: track 78.6 -> 105.3 mm
- net A11: track 46.4 -> 72.3 mm
- net D2: track 190.9 -> 216.6 mm
- net A10: track 47.2 -> 68.6 mm, vias 1 -> 0
- net A3: track 74.7 -> 96.1 mm
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Other:
- board size 200 x 100 mm -> 280 x 140 mm

Commit message: feat(kicad): re-route led/cf/control/io with right-edge LED banks
Status LEDs now on the edge opposite the connector; re-routed at 280x140.
0 unconnected on all four.

Co-Authored-By: Claude Opus 4.8 <noreply@anthropic.com>
Parts:
- moved RP1 30.5 mm to (250.9, 13.3)
- moved R4 19.2 mm to (250.9, 23.8)
- moved LED3 16.2 mm to (272.3, 13.3), turned to 180 degrees
- moved LED4 13.3 mm to (272.3, 23.8), turned to 180 degrees
Routing:
- net D5: track 197.7 -> 219.2 mm, vias 2 -> 1
- net LEDP: track 29.2 -> 8.65 mm
- net D0: track 187.9 -> 207.5 mm, vias 0 -> 1
- net A2: track 100.4 -> 115.4 mm
- net LEDWR: track 22.9 -> 8.65 mm
- net D7: track 186.9 -> 201.1 mm
- net A9: track 86.7 -> 98.8 mm
- net A10: track 68.6 -> 80.6 mm, vias 0 -> 1
- net D1: track 200.1 -> 211.4 mm
- net D6: track 193.2 -> 203.7 mm
- net LP5: track 52.8 -> 61.5 mm, vias 0 -> 1
- net LP6: track 57.4 -> 65.6 mm
- net D3: track 214.8 -> 222.4 mm
- net LR4: track 22.6 -> 29.2 mm
- net A12: track 64.4 -> 70.8 mm
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