File: hardware/memory-card/kicad/p8x-memory-card.kicad_pcb (KiCad board)
At the start: 4 copper layers, 280 x 140 mm, 36 parts, among them J1 MABC96R, U1 28C256, U10 62256, U11 74HCT32, U2 62256, U3 74HCT245, U4 74HCT30, U5 74HCT138, U6 74HCT138, U7 74HCT00, U8 74HCT32, U9 74HCT08

Commit message: feat(kicad): memory card LED order PWR/ROM/RAML/RAMH/RD/WR (rework)
Reorder the right-edge status LEDs top-to-bottom to PWR, ROM, RAML, RAMH, RD,
WR (was PWR, ROM, RAMH, RD, WR, RAML). Each LEDPAIR tuple keeps its
(resistor, LED, function) pairing -- only the row position + silk label move.
Re-routed: 920 tracks, 41 vias, DRC 0 violations (the 1 pre-existing LEDRA
unconnected persists). Gerbers/render/placement regenerated.

Co-Authored-By: Claude Opus 4.8 <noreply@anthropic.com>
Parts:
- moved LED7 42.0 mm to (272.3, 58.0)
- moved RS5 42.0 mm to (244.9, 58.0)
- moved LED4 14.0 mm to (272.3, 72.0)
- moved LED5 14.0 mm to (272.3, 86.0)
- moved LED6 14.0 mm to (272.3, 100.0)
- moved RS2 14.0 mm to (244.9, 72.0)
- moved RS3 14.0 mm to (244.9, 86.0)
- moved RS4 14.0 mm to (244.9, 100.0)
Routing:
- net A2: track 180.1 -> 223.5 mm
- net A0: track 191.0 -> 227.4 mm, vias 2 -> 1
- net A3: track 176.9 -> 206.3 mm, vias 2 -> 0
- net -RD: track 248.0 -> 224.2 mm
- net D0: track 64.7 -> 84.8 mm, vias 0 -> 1
- net A4: track 175.5 -> 195.3 mm
- net A1: track 188.1 -> 207.4 mm, vias 2 -> 1
- net LEDRA2: track 14.7 -> 0.00 mm
- net LEDRA: track 0.00 -> 14.7 mm
- net D4: track 62.4 -> 76.1 mm
- net A10: track 224.8 -> 211.3 mm, vias 1 -> 0
- net DLD1: track 145.0 -> 132.2 mm, vias 0 -> 1
- net DOE1: track 94.3 -> 104.0 mm
- net A8: track 202.6 -> 211.5 mm
- net MD2: track 128.1 -> 119.3 mm
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
Commit message: fix(memory-card): stitch the last LED-bank net -> DRC fully clean
Freerouting left LEDRA2 (RS5->LED7, the RAML LED) unrouted because the direct
top-layer path is blocked by the ROMK track. import_ses.py now self-heals: any
trivial 2-pad net left with no copper and collinear pads gets a straight B.Cu
track (through-hole pads let it duck under the F.Cu tracks). Memory card DRC is
now 0 violations, 0 unconnected (was 1 unconnected). Gerbers/render regenerated.

Co-Authored-By: Claude Opus 4.8 <noreply@anthropic.com>
Routing:
- net LEDRA2: track 0.00 -> 14.7 mm

Commit message: feat(memory-card): one-command build+verify; fix the wx.App exit hang
Add hardware/memory-card/kicad/build.sh: from the (deterministic) placement +
netlist it re-runs PCB trace layout (Freerouting) -> import + self-heal stitch
-> gerbers/drill/render -> the full check (ERC + gate-sim + DRC + keepout + fab),
ending in a PASS/FAIL verdict. Ran end-to-end in ~90s, memory card PASS.

Fix the wx.App exit hang that made the pipeline scripts need babysitting:
kicad_tools.py, export_dsn.py and import_ses.py now os._exit(0) after saving, so
they terminate instead of blocking on the wx event loop. This is what makes the
build fully scriptable. Board is a fresh route from the same placement.

Co-Authored-By: Claude Opus 4.8 <noreply@anthropic.com>
Routing:
- net D1: track 64.5 -> 85.9 mm
- net A0: track 227.4 -> 207.0 mm
- net A2: track 223.5 -> 241.9 mm, vias 1 -> 2
- net A5: track 170.4 -> 185.7 mm, vias 1 -> 0
- net D4: track 76.1 -> 62.5 mm
- net A3: track 206.3 -> 197.5 mm, vias 0 -> 1
- net MD7: track 136.2 -> 144.2 mm, vias 2 -> 0
- net A1: track 207.4 -> 214.6 mm, vias 1 -> 3
- net DOE2: track 97.5 -> 104.3 mm, vias 2 -> 1
- net D0: track 84.8 -> 78.1 mm, vias 1 -> 3
- net A14: track 237.2 -> 231.3 mm
- net -WE: track 176.3 -> 170.6 mm, vias 2 -> 3
- net A8: track 211.5 -> 206.4 mm
- net -RD: track 224.2 -> 229.2 mm, vias 0 -> 2
- net RDK: track 136.6 -> 140.5 mm, vias 0 -> 1
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
Commit message: build: re-route all boards via the build+verify flow (keepouts + stitch)
Ran build.sh all + build.sh backplane. Every board regenerated + re-routed fresh
with the mounting-hole keepouts, the self-heal stitch, and -mt 1. Final verdicts:
  PASS (clean): cf, control, alu, regbank, memory
  1 unconnected net (non-collinear, stitch gap): io, peripheral
  18 unconnected (dense ~960-pin bus, router cap): backplane
  3 blocking DRC: bustest
All boards now PASS the DIN mounting-hole keepout check; 0 blocking DRC except
bustest. Gerbers/renders/placement + DRC reports regenerated per card.

Co-Authored-By: Claude Opus 4.8 <noreply@anthropic.com>
Routing:
- net A2: track 241.9 -> 195.3 mm, vias 2 -> 1
- net -RD: track 229.2 -> 255.4 mm, vias 2 -> 1
- net D1: track 85.9 -> 62.5 mm, vias 1 -> 0
- net D4: track 62.5 -> 81.9 mm, vias 1 -> 0
- net A4: track 191.9 -> 174.0 mm, vias 1 -> 0
- net -WE: track 170.6 -> 188.5 mm, vias 3 -> 0
- net A1: track 214.6 -> 197.8 mm, vias 3 -> 1
- net MD5: track 130.5 -> 147.2 mm, vias 1 -> 0
- net A5: track 185.7 -> 170.0 mm
- net DLD2: track 134.6 -> 149.0 mm
- net D0: track 78.1 -> 64.8 mm, vias 3 -> 0
- net A14: track 231.3 -> 244.5 mm
- net A11: track 284.5 -> 271.4 mm, vias 1 -> 0
- net A3: track 197.5 -> 184.5 mm
- net ROMCE: track 166.2 -> 154.0 mm
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