File: hardware/peripheral-card/kicad/p8x-peripheral-card.kicad_pcb (KiCad board)
At the start: 4 copper layers, 280 x 140 mm, 104 parts, among them J1 MABC96R, J3 1x3, J4 IDE-40, SW1 INPUT, U1 74HCT30, U10 74HCT374, U11 74HCT244, U12 74HCT244, U13 74HCT244, U14 6850, U15 74HCT00, U16 DS1302, U17 74HCT245, U18 74HCT14, U19 74HCT10, U2 74HCT138, U20 74HCT10, U21 74HCT08, U22 74HCT374, U23 6850, U24 PS/2 MCU, U25 WIN CMP, U26 74HCT138, U27 74HCT138, U28 74HCT374, U29 74HCT374, U3 74HCT138, U30 74HCT374, U31 74HCT374, U32 74HCT244, U33 74HCT244, U4 74HCT138, U5 74HCT32, U6 74HCT08, U7 74HCT161, U8 MAX232, U9 74HCT244, X2 2.4576MHZ, X3 32.768KHZ

Commit message: feat(peripheral-card): stage 3 route -- 6150 tracks, DRC-clean
Freerouting completed the 33-IC combined card: 6150 tracks, 365 vias. DRC = 4
violations (all cosmetic silk-edge-clearance) + 2 unconnected nets; the DIN
mounting-hole keepout is respected (0 tracks within 4mm). Gerbers/drill/zip +
top render generated; build artifacts gitignored. Also commit the memory-card
gerbers regenerated by the LED-reorder rework.

Co-Authored-By: Claude Opus 4.8 <noreply@anthropic.com>
Routing:
- net D0: track 0.00 -> 499.2 mm, vias 0 -> 5
- net D1: track 0.00 -> 465.4 mm, vias 0 -> 4
- net D6: track 0.00 -> 460.9 mm, vias 0 -> 8
- net D2: track 0.00 -> 456.1 mm, vias 0 -> 6
- net D4: track 0.00 -> 453.3 mm, vias 0 -> 9
- net D3: track 0.00 -> 446.5 mm, vias 0 -> 4
- net A1: track 0.00 -> 425.7 mm, vias 0 -> 2
- net D5: track 0.00 -> 418.5 mm, vias 0 -> 2
- net A0: track 0.00 -> 415.7 mm, vias 0 -> 4
- net D7: track 0.00 -> 407.2 mm, vias 0 -> 5
- net A2: track 0.00 -> 397.5 mm, vias 0 -> 5
- net A3: track 0.00 -> 370.0 mm, vias 0 -> 9
- net MB5: track 0.00 -> 363.0 mm, vias 0 -> 5
- net MB3: track 0.00 -> 338.9 mm, vias 0 -> 3
- net MB4: track 0.00 -> 336.9 mm, vias 0 -> 2
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
Commit message: build: re-route all boards via the build+verify flow (keepouts + stitch)
Ran build.sh all + build.sh backplane. Every board regenerated + re-routed fresh
with the mounting-hole keepouts, the self-heal stitch, and -mt 1. Final verdicts:
  PASS (clean): cf, control, alu, regbank, memory
  1 unconnected net (non-collinear, stitch gap): io, peripheral
  18 unconnected (dense ~960-pin bus, router cap): backplane
  3 blocking DRC: bustest
All boards now PASS the DIN mounting-hole keepout check; 0 blocking DRC except
bustest. Gerbers/renders/placement + DRC reports regenerated per card.

Co-Authored-By: Claude Opus 4.8 <noreply@anthropic.com>
Routing:
- net SIN2: track 148.5 -> 292.6 mm
- net VBAT: track 0.00 -> 139.0 mm, vias 0 -> 2
- net SIN: track 159.6 -> 236.2 mm, vias 0 -> 7
- net RDP: track 287.3 -> 228.7 mm, vias 3 -> 1
- net MA10: track 158.5 -> 103.4 mm, vias 7 -> 4
- net RTCX2: track 155.5 -> 202.6 mm
- net VMN: track 290.5 -> 245.6 mm, vias 5 -> 6
- net MA12: track 109.9 -> 151.5 mm, vias 2 -> 5
- net D0: track 499.2 -> 458.9 mm, vias 5 -> 8
- net MA8: track 104.6 -> 144.8 mm, vias 1 -> 3
- net -IOR: track 272.3 -> 309.1 mm, vias 3 -> 5
- net A1: track 425.7 -> 389.7 mm, vias 2 -> 3
- net D5: track 418.5 -> 453.6 mm, vias 2 -> 9
- net A3: track 370.0 -> 335.0 mm, vias 9 -> 2
- net -RR4: track 96.6 -> 131.3 mm, vias 0 -> 1
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