File: hardware/regbank-card/kicad/p8x-regbank-card.kicad_pcb (KiCad board)
At the start: 4 copper layers, 340 x 100 mm, 95 parts, among them J1 MABC96R, U1 74HCT169, U10 74HCT169, U11 74HCT169, U12 74HCT169, U13 74HCT169, U14 74HCT169, U15 74HCT169, U16 74HCT169, U17 74HCT244, U18 74HCT244, U19 74HCT244, U2 74HCT169, U20 74HCT244, U21 74HCT244, U22 74HCT244, U23 74HCT244, U24 74HCT244, U25 74HCT244, U26 74HCT244, U27 74HCT257, U28 74HCT257, U29 74HCT244, U3 74HCT169, U30 74HCT138, U31 74HCT138, U32 74HCT139, U33 74HCT138, U34 74HCT02, U35 74HCT14, U36 74HCT244, U37 74HCT08, U38 74HCT08, U39 74HCT139, U4 74HCT169, U40 74HCT32, U41 74HCT377, U42 74HCT377, U43 74HCT244, U44 74HCT244, U5 74HCT169, U6 74HCT169, U7 74HCT169, U8 74HCT169, U9 74HCT169

Commit message: feat(kicad): uniform 280x140 -- memory re-routed; regbank/bustest placed
memory-card re-routed at the uniform 280x140 (986 tracks, 0 violations). regbank
+ bustest placed at 280x140 with clean placement + planes but routing pending
(densest boards exceeded Freerouting's time budget). Status doc updated; PS/2
level-shift noted as NOYITO TXS0102.

Co-Authored-By: Claude Opus 4.8 <noreply@anthropic.com>
Parts:
- moved RP1 263.3 mm to (64.1, 103.6)
- moved R4 242.3 mm to (81.4, 103.6)
- moved C44 237.9 mm to (42.5, 104.7)
- moved U44 237.9 mm to (33.6, 116.8)
- moved LED3 235.5 mm to (117.0, 105.4), turned to 0 degrees
- moved R5 221.5 mm to (98.8, 103.6)
- moved LED4 219.6 mm to (128.6, 105.4), turned to 0 degrees
- moved C34 217.1 mm to (256.1, 67.1)
- moved U34 217.1 mm to (251.0, 79.2)
- moved U10 206.4 mm to (33.6, 41.5)
- moved C10 206.4 mm to (40.0, 29.4)
- moved LED5 204.0 mm to (140.1, 105.4), turned to 0 degrees
- moved U11 203.3 mm to (59.5, 41.5)
- moved C11 203.3 mm to (65.9, 29.4)
- moved C12 200.1 mm to (91.8, 29.4)
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Routing:
- net D5: track 562.7 -> 0.00 mm, vias 9 -> 0
- net D4: track 557.9 -> 0.00 mm, vias 7 -> 0
- net D7: track 555.7 -> 0.00 mm, vias 10 -> 0
- net D3: track 549.7 -> 0.00 mm, vias 7 -> 0
- net D2: track 542.8 -> 0.00 mm, vias 9 -> 0
- net D6: track 529.0 -> 0.00 mm, vias 10 -> 0
- net D1: track 523.0 -> 0.00 mm, vias 6 -> 0
- net D0: track 515.8 -> 0.00 mm, vias 4 -> 0
- net CLK: track 489.3 -> 0.00 mm, vias 2 -> 0
- net UDB: track 411.2 -> 0.00 mm, vias 5 -> 0
- net PSEL1: track 359.2 -> 0.00 mm, vias 2 -> 0
- net PSEL0: track 350.4 -> 0.00 mm, vias 2 -> 0
- net PSEL2: track 338.6 -> 0.00 mm, vias 1 -> 0
- net PB2: track 310.1 -> 0.00 mm, vias 4 -> 0
- net PB15: track 309.7 -> 0.00 mm, vias 7 -> 0
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Other:
- board size 340 x 100 mm -> 280 x 140 mm

Commit message: feat(kicad): regbank-card fully routed at 280x140 (right-edge LEDs)
The new right-edge-LED layout auto-routed in 5m45s (vs 10min before); the slow
single-threaded optimizer pass then completed (~13min). 4089 tracks, 213 vias,
0 unconnected. Densest card, so cosmetic silk crowding remains.

Co-Authored-By: Claude Opus 4.8 <noreply@anthropic.com>
Parts:
- moved C9 208.1 mm to (40.0, 29.4)
- moved U9 208.1 mm to (33.6, 41.5)
- moved RP1 207.6 mm to (250.9, 13.3)
- moved R4 187.4 mm to (250.9, 23.8)
- moved C17 182.3 mm to (42.5, 48.2)
- moved C18 182.3 mm to (73.5, 48.2)
- moved U17 182.3 mm to (33.6, 60.4)
- moved U18 182.3 mm to (64.6, 60.4)
- moved LED3 180.5 mm to (272.3, 13.3), turned to 180 degrees
- moved R5 167.2 mm to (250.9, 34.3)
- moved LED4 165.3 mm to (272.3, 23.8), turned to 180 degrees
- moved C24 156.1 mm to (42.5, 67.1)
- moved C25 156.1 mm to (73.5, 67.1)
- moved U24 156.1 mm to (33.6, 79.2)
- moved U25 156.1 mm to (64.6, 79.2)
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Routing:
- net D4: track 0.00 -> 531.0 mm, vias 0 -> 3
- net D6: track 0.00 -> 523.7 mm, vias 0 -> 3
- net D5: track 0.00 -> 513.8 mm, vias 0 -> 4
- net D7: track 0.00 -> 511.6 mm, vias 0 -> 4
- net D3: track 0.00 -> 500.2 mm, vias 0 -> 8
- net D0: track 0.00 -> 495.5 mm, vias 0 -> 1
- net CLK: track 0.00 -> 494.5 mm, vias 0 -> 1
- net D1: track 0.00 -> 494.4 mm, vias 0 -> 3
- net D2: track 0.00 -> 491.7 mm, vias 0 -> 2
- net UDB: track 0.00 -> 414.4 mm, vias 0 -> 2
- net PB2: track 0.00 -> 346.1 mm, vias 0 -> 4
- net PB1: track 0.00 -> 338.6 mm, vias 0 -> 4
- net PB3: track 0.00 -> 326.2 mm, vias 0 -> 4
- net PB0: track 0.00 -> 322.6 mm, vias 0 -> 6
- net PB8: track 0.00 -> 316.8 mm, vias 0 -> 2
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
Commit message: build: re-route all boards via the build+verify flow (keepouts + stitch)
Ran build.sh all + build.sh backplane. Every board regenerated + re-routed fresh
with the mounting-hole keepouts, the self-heal stitch, and -mt 1. Final verdicts:
  PASS (clean): cf, control, alu, regbank, memory
  1 unconnected net (non-collinear, stitch gap): io, peripheral
  18 unconnected (dense ~960-pin bus, router cap): backplane
  3 blocking DRC: bustest
All boards now PASS the DIN mounting-hole keepout check; 0 blocking DRC except
bustest. Gerbers/renders/placement + DRC reports regenerated per card.

Co-Authored-By: Claude Opus 4.8 <noreply@anthropic.com>
Routing:
- net -LDH0E: track 228.1 -> 186.5 mm, vias 1 -> 3
- net -LDH2: track 136.3 -> 96.7 mm, vias 1 -> 0
- net -LDL0E: track 230.8 -> 269.1 mm, vias 3 -> 1
- net D1: track 494.4 -> 526.8 mm, vias 3 -> 5
- net PB13: track 289.4 -> 259.1 mm, vias 3 -> 5
- net PB10: track 274.9 -> 304.9 mm
- net D0: track 495.5 -> 524.7 mm, vias 1 -> 2
- net PINC: track 160.0 -> 131.8 mm, vias 2 -> 1
- net -LDL3: track 186.4 -> 160.8 mm, vias 4 -> 1
- net PB5: track 268.9 -> 294.4 mm, vias 4 -> 2
- net A0: track 78.0 -> 103.2 mm, vias 1 -> 2
- net PQ2_0: track 159.1 -> 134.2 mm, vias 1 -> 0
- net PB1: track 338.6 -> 314.3 mm
- net -SEL0: track 96.6 -> 120.7 mm
- net PQ1_4: track 99.1 -> 75.4 mm
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