File: hardware/regbank-card/kicad/p8x-regbank-card-1.kicad_sch (KiCad schematic)
At the start: 9 parts, among them U1 74HCT169, U2 74HCT169, U3 74HCT169, U4 74HCT169, U5 74HCT169, U6 74HCT169, U7 74HCT169, U8 74HCT169, U9 74HCT169

Commit message: feat(sch): draw every P8X card schematic by function
Extend the functional-sheet grouping from the io-card to the control,
regbank, alu, memory, cf, ps2 and bustest cards. functional_sheets now
attaches unnamed glue gates, LEDs, resistors and connectors to the block
they share the most local nets with, so each block lists only its main
parts. A net with two or more pins on a sheet is now wired there even if
it continues elsewhere (its global name label rides on the wire), and
every wire is oriented by drawing side. The regbank gets one pointer per
sheet; the ps2 latches share a sheet with the AVR so the mailbox bus is
drawn. The bustest probe resistors use a straight-order RNISO8DSTR
drawing (the reversed B side forced every wire to cross and the sheet
fell back to labels). build_sch.sh now shows ELK fallbacks and clears old
numbered sheets before a build. All eight netlists match the boards,
ERC 0 errors; the boards change only in footprint link paths.

Co-Authored-By: Claude Opus 5.5 <noreply@anthropic.com>
Parts:
- removed U5, U6, U7, U8, U9: 74HCT169, Package_DIP:DIP-16_W7.62mm, symbol p8x:74169
- added U17, U18: 74HCT244, Package_DIP:DIP-20_W7.62mm, symbol p8x:74244
Connections:
- net GND: now also U17.10, U18.10
- net PQ0_0: now also U17.2 (A1)
- net PQ0_1: now also U17.4 (A2)
- net PQ0_10: now also U18.6 (A3)
- net PQ0_11: now also U18.8 (A4)
- net PQ0_12: now also U18.11 (A5)
- net PQ0_13: now also U18.13 (A6)
- net PQ0_14: now also U18.15 (A7)
- net PQ0_15: now also U18.17 (A8)
- net PQ0_2: now also U17.6 (A3)
- net PQ0_3: now also U17.8 (A4)
- net PQ0_4: now also U17.11 (A5)
- net PQ0_5: now also U17.13 (A6)
- net PQ0_6: now also U17.15 (A7)
- net PQ0_7: now also U17.17 (A8)
- net PQ0_8: now also U18.2 (A1)
- net PQ0_9: now also U18.4 (A2)
- net VCC: now also U17.20, U18.20
- new net -SEL0: U17.1 (!G1), U17.19 (!G2), U18.1 (!G1), U18.19 (!G2)
- new net PB0: U17.18 (Y1)
- new net PB1: U17.16 (Y2)
- new net PB10: U18.14 (Y3)
- new net PB11: U18.12 (Y4)
- new net PB12: U18.9 (Y5)
- new net PB13: U18.7 (Y6)
- new net PB14: U18.5 (Y7)
- new net PB15: U18.3 (Y8)
- new net PB2: U17.14 (Y3)
- new net PB3: U17.12 (Y4)
- new net PB4: U17.9 (Y5)
- new net PB5: U17.7 (Y6)
- new net PB6: U17.5 (Y7)
- new net PB7: U17.3 (Y8)
- new net PB8: U18.18 (Y1)
- new net PB9: U18.16 (Y2)
- no-connect marks 2 -> 1
Other:
- moved on the sheet: U1, U2, U3, U4
