File: hardware/regbank-card/kicad/p8x-regbank-card-3.kicad_sch (KiCad schematic)
At the start: 9 parts, among them U19 74HCT244, U20 74HCT244, U21 74HCT244, U22 74HCT244, U23 74HCT244, U24 74HCT244, U25 74HCT244, U26 74HCT244, U27 74HCT257

Commit message: feat(sch): draw every P8X card schematic by function
Extend the functional-sheet grouping from the io-card to the control,
regbank, alu, memory, cf, ps2 and bustest cards. functional_sheets now
attaches unnamed glue gates, LEDs, resistors and connectors to the block
they share the most local nets with, so each block lists only its main
parts. A net with two or more pins on a sheet is now wired there even if
it continues elsewhere (its global name label rides on the wire), and
every wire is oriented by drawing side. The regbank gets one pointer per
sheet; the ps2 latches share a sheet with the AVR so the mailbox bus is
drawn. The bustest probe resistors use a straight-order RNISO8DSTR
drawing (the reversed B side forced every wire to cross and the sheet
fell back to labels). build_sch.sh now shows ELK fallbacks and clears old
numbered sheets before a build. All eight netlists match the boards,
ERC 0 errors; the boards change only in footprint link paths.

Co-Authored-By: Claude Opus 5.5 <noreply@anthropic.com>
Parts:
- removed U19, U20, U23, U24, U25, U26: 74HCT244, Package_DIP:DIP-20_W7.62mm, symbol p8x:74244
- removed U27: 74HCT257, Package_DIP:DIP-16_W7.62mm, symbol p8x:74257
- added U10, U11, U12, U9: 74HCT169, Package_DIP:DIP-16_W7.62mm, symbol p8x:74169
Connections:
- net GND: now also U10.8, U11.8, U12.8, U9.10 (!ENT), U9.8
- net PQ2_0: now also U9.14 (QA)
- net PQ2_1: now also U9.13 (QB)
- net PQ2_10: now also U11.12 (QC)
- net PQ2_11: now also U11.11 (QD)
- net PQ2_12: now also U12.14 (QA)
- net PQ2_13: now also U12.13 (QB)
- net PQ2_14: now also U12.12 (QC)
- net PQ2_15: now also U12.11 (QD)
- net PQ2_2: now also U9.12 (QC)
- net PQ2_3: now also U9.11 (QD)
- net PQ2_4: now also U10.14 (QA)
- net PQ2_5: now also U10.13 (QB)
- net PQ2_6: now also U10.12 (QC)
- net PQ2_7: now also U10.11 (QD)
- net PQ2_8: now also U11.14 (QA)
- net PQ2_9: now also U11.13 (QB)
- net VCC: now also U10.16, U11.16, U12.16, U9.16
- new net -CNT2: U10.7 (!ENP), U11.7 (!ENP), U12.7 (!ENP), U9.7 (!ENP)
- new net -LDH2: U11.9 (!LOAD), U12.9 (!LOAD)
- new net -LDL2: U10.9 (!LOAD), U9.9 (!LOAD)
- new net CLK: U10.2 (CLK), U11.2 (CLK), U12.2 (CLK), U9.2 (CLK)
- new net D0: U11.3 (A), U9.3 (A)
- new net D1: U11.4 (B), U9.4 (B)
- new net D2: U11.5 (C), U9.5 (C)
- new net D3: U11.6 (D), U9.6 (D)
- new net D4: U10.3 (A), U12.3 (A)
- new net D5: U10.4 (B), U12.4 (B)
- new net D6: U10.5 (C), U12.5 (C)
- new net D7: U10.6 (D), U12.6 (D)
- new net RC2_0: U10.10 (!ENT), U9.15 (!RCO)
- new net RC2_1: U10.15 (!RCO), U11.10 (!ENT)
- new net RC2_2: U11.15 (!RCO), U12.10 (!ENT)
- new net UDB: U10.1 (UD), U11.1 (UD), U12.1 (UD), U9.1 (UD)
- no-connect marks 0 -> 1
Other:
- moved on the sheet: U21, U22
