File: hardware/regbank-card/kicad/p8x-regbank-card-4.kicad_sch (KiCad schematic)
At the start: 9 parts, among them U28 74HCT257, U29 74HCT244, U30 74HCT138, U31 74HCT138, U32 74HCT139, U33 74HCT138, U34 74HCT02, U35 74HCT14, U36 74HCT244

Commit message: feat(sch): draw every P8X card schematic by function
Extend the functional-sheet grouping from the io-card to the control,
regbank, alu, memory, cf, ps2 and bustest cards. functional_sheets now
attaches unnamed glue gates, LEDs, resistors and connectors to the block
they share the most local nets with, so each block lists only its main
parts. A net with two or more pins on a sheet is now wired there even if
it continues elsewhere (its global name label rides on the wire), and
every wire is oriented by drawing side. The regbank gets one pointer per
sheet; the ps2 latches share a sheet with the AVR so the mailbox bus is
drawn. The bustest probe resistors use a straight-order RNISO8DSTR
drawing (the reversed B side forced every wire to cross and the sheet
fell back to labels). build_sch.sh now shows ELK fallbacks and clears old
numbered sheets before a build. All eight netlists match the boards,
ERC 0 errors; the boards change only in footprint link paths.

Co-Authored-By: Claude Opus 5.5 <noreply@anthropic.com>
Parts:
- removed U28: 74HCT257, Package_DIP:DIP-16_W7.62mm, symbol p8x:74257
- removed U29, U36: 74HCT244, Package_DIP:DIP-20_W7.62mm, symbol p8x:74244
- removed U30, U31, U33: 74HCT138, Package_DIP:DIP-16_W7.62mm, symbol p8x:74138
- removed U32: 74HCT139, Package_DIP:DIP-16_W7.62mm, symbol p8x:74139
- removed U34: 74HCT02, Package_DIP:DIP-14_W7.62mm, symbol p8x:7402
- removed U35: 74HCT14, Package_DIP:DIP-14_W7.62mm, symbol p8x:HEX14
- added U13, U14, U15, U16: 74HCT169, Package_DIP:DIP-16_W7.62mm, symbol p8x:74169
- added U23, U24: 74HCT244, Package_DIP:DIP-20_W7.62mm, symbol p8x:74244
Connections:
- net -LDH3: now also U15.9 (!LOAD), U16.9 (!LOAD)
- net -LDL3: now also U13.9 (!LOAD), U14.9 (!LOAD)
- net -SEL3: now also U23.1 (!G1), U23.19 (!G2), U24.1 (!G1), U24.19 (!G2)
- net D0: now also U13.3 (A), U15.3 (A)
- net D1: now also U13.4 (B), U15.4 (B)
- net D2: now also U13.5 (C), U15.5 (C)
- net D3: now also U13.6 (D), U15.6 (D)
- net D4: now also U14.3 (A), U16.3 (A)
- net D5: now also U14.4 (B), U16.4 (B)
- net D6: now also U14.5 (C), U16.5 (C)
- net D7: now also U14.6 (D), U16.6 (D)
- net GND: now also U13.10 (!ENT), U13.8, U14.8, U15.8, U16.8, U23.10, U24.10
- net PB12: now also U24.9 (Y5)
- net PB13: now also U24.7 (Y6)
- net PB14: now also U24.5 (Y7)
- net PB15: now also U24.3 (Y8)
- net PB4: now also U23.9 (Y5)
- net PB5: now also U23.7 (Y6)
- net PB6: now also U23.5 (Y7)
- net PB7: now also U23.3 (Y8)
- net UDB: now also U13.1 (UD), U14.1 (UD), U15.1 (UD), U16.1 (UD)
- net VCC: now also U13.16, U14.16, U15.16, U16.16, U23.20, U24.20
- new net -CNT3: U13.7 (!ENP), U14.7 (!ENP), U15.7 (!ENP), U16.7 (!ENP)
- new net CLK: U13.2 (CLK), U14.2 (CLK), U15.2 (CLK), U16.2 (CLK)
- new net PB0: U23.18 (Y1)
- new net PB1: U23.16 (Y2)
- new net PB10: U24.14 (Y3)
- new net PB11: U24.12 (Y4)
- new net PB2: U23.14 (Y3)
- new net PB3: U23.12 (Y4)
- new net PB8: U24.18 (Y1)
- new net PB9: U24.16 (Y2)
- new net PQ3_0: U13.14 (QA), U23.2 (A1)
- new net PQ3_1: U13.13 (QB), U23.4 (A2)
- new net PQ3_10: U15.12 (QC), U24.6 (A3)
- new net PQ3_11: U15.11 (QD), U24.8 (A4)
- new net PQ3_12: U16.14 (QA), U24.11 (A5)
- new net PQ3_13: U16.13 (QB), U24.13 (A6)
- new net PQ3_14: U16.12 (QC), U24.15 (A7)
- new net PQ3_15: U16.11 (QD), U24.17 (A8)
- new net PQ3_2: U13.12 (QC), U23.6 (A3)
- new net PQ3_3: U13.11 (QD), U23.8 (A4)
- new net PQ3_4: U14.14 (QA), U23.11 (A5)
- new net PQ3_5: U14.13 (QB), U23.13 (A6)
- new net PQ3_6: U14.12 (QC), U23.15 (A7)
- new net PQ3_7: U14.11 (QD), U23.17 (A8)
- new net PQ3_8: U15.14 (QA), U24.2 (A1)
- new net PQ3_9: U15.13 (QB), U24.4 (A2)
- new net RC3_0: U13.15 (!RCO), U14.10 (!ENT)
- new net RC3_1: U14.15 (!RCO), U15.10 (!ENT)
- new net RC3_2: U15.15 (!RCO), U16.10 (!ENT)
- no-connect marks 21 -> 1
