File: hardware/regbank-card/kicad/p8x-regbank-card-7.kicad_sch (KiCad schematic)
At the start: 1 part, among them J1 MABC96R

Commit message: feat(sch): draw every P8X card schematic by function
Extend the functional-sheet grouping from the io-card to the control,
regbank, alu, memory, cf, ps2 and bustest cards. functional_sheets now
attaches unnamed glue gates, LEDs, resistors and connectors to the block
they share the most local nets with, so each block lists only its main
parts. A net with two or more pins on a sheet is now wired there even if
it continues elsewhere (its global name label rides on the wire), and
every wire is oriented by drawing side. The regbank gets one pointer per
sheet; the ps2 latches share a sheet with the AVR so the mailbox bus is
drawn. The bustest probe resistors use a straight-order RNISO8DSTR
drawing (the reversed B side forced every wire to cross and the sheet
fell back to labels). build_sch.sh now shows ELK fallbacks and clears old
numbered sheets before a build. All eight netlists match the boards,
ERC 0 errors; the boards change only in footprint link paths.

Co-Authored-By: Claude Opus 5.5 <noreply@anthropic.com>
Parts:
- removed J1: MABC96R, Connector_DIN:DIN41612_C_3x32_Male_Horizontal_THT, symbol p8x:DIN96C
- added U25, U26, U29: 74HCT244, Package_DIP:DIP-20_W7.62mm, symbol p8x:74244
- added U27, U28: 74HCT257, Package_DIP:DIP-16_W7.62mm, symbol p8x:74257
Connections:
- net A0: now also U25.18 (Y1)
- net A1: now also U25.16 (Y2)
- net A10: now also U26.14 (Y3)
- net A11: now also U26.12 (Y4)
- net A12: now also U26.9 (Y5)
- net A13: now also U26.7 (Y6)
- net A14: now also U26.5 (Y7)
- net A15: now also U26.3 (Y8)
- net A2: now also U25.14 (Y3)
- net A3: now also U25.12 (Y4)
- net A4: now also U25.9 (Y5)
- net A5: now also U25.7 (Y6)
- net A6: now also U25.5 (Y7)
- net A7: now also U25.3 (Y8)
- net A8: now also U26.18 (Y1)
- net A9: now also U26.16 (Y2)
- net D0: now also U29.18 (Y1)
- net D1: now also U29.16 (Y2)
- net D2: now also U29.14 (Y3)
- net D3: now also U29.12 (Y4)
- net D4: now also U29.9 (Y5)
- net D5: now also U29.7 (Y6)
- net D6: now also U29.5 (Y7)
- net D7: now also U29.3 (Y8)
- net GND: now also U25.1 (!G1), U25.10, U25.19 (!G2), U26.1 (!G1), U26.10, U26.19 (!G2), U27.15 (!OE), U27.8, U28.15 (!OE), U28.8, U29.10
- net VCC: now also U25.20, U26.20, U27.16, U28.16, U29.20
- new net -POE: U29.1 (!G1), U29.19 (!G2)
- new net PB0: U25.2 (A1), U27.2 (A1)
- new net PB1: U25.4 (A2), U27.5 (A2)
- new net PB10: U26.6 (A3), U27.10 (B3)
- new net PB11: U26.8 (A4), U27.13 (B4)
- new net PB12: U26.11 (A5), U28.3 (B1)
- new net PB13: U26.13 (A6), U28.6 (B2)
- new net PB14: U26.15 (A7), U28.10 (B3)
- new net PB15: U26.17 (A8), U28.13 (B4)
- new net PB2: U25.6 (A3), U27.11 (A3)
- new net PB3: U25.8 (A4), U27.14 (A4)
- new net PB4: U25.11 (A5), U28.2 (A1)
- new net PB5: U25.13 (A6), U28.5 (A2)
- new net PB6: U25.15 (A7), U28.11 (A3)
- new net PB7: U25.17 (A8), U28.14 (A4)
- new net PB8: U26.2 (A1), U27.3 (B1)
- new net PB9: U26.4 (A2), U27.6 (B2)
- new net POEHP: U27.1 (S), U28.1 (S)
- new net RB0: U27.4 (Y1), U29.2 (A1)
- new net RB1: U27.7 (Y2), U29.4 (A2)
- new net RB2: U27.9 (Y3), U29.6 (A3)
- new net RB3: U27.12 (Y4), U29.8 (A4)
- new net RB4: U28.4 (Y1), U29.11 (A5)
- new net RB5: U28.7 (Y2), U29.13 (A6)
- new net RB6: U28.9 (Y3), U29.15 (A7)
- new net RB7: U28.12 (Y4), U29.17 (A8)
- no-connect marks 33 -> 0
