File: hardware/regbank-card/kicad/p8x-regbank-card-8.kicad_sch (KiCad schematic)
At the start: 59 parts

Commit message: feat(sch): draw every P8X card schematic by function
Extend the functional-sheet grouping from the io-card to the control,
regbank, alu, memory, cf, ps2 and bustest cards. functional_sheets now
attaches unnamed glue gates, LEDs, resistors and connectors to the block
they share the most local nets with, so each block lists only its main
parts. A net with two or more pins on a sheet is now wired there even if
it continues elsewhere (its global name label rides on the wire), and
every wire is oriented by drawing side. The regbank gets one pointer per
sheet; the ps2 latches share a sheet with the AVR so the mailbox bus is
drawn. The bustest probe resistors use a straight-order RNISO8DSTR
drawing (the reversed B side forced every wire to cross and the sheet
fell back to labels). build_sch.sh now shows ELK fallbacks and clears old
numbered sheets before a build. All eight netlists match the boards,
ERC 0 errors; the boards change only in footprint link paths.

Co-Authored-By: Claude Opus 5.5 <noreply@anthropic.com>
Parts:
- removed C1, C10, C11, C12, C13, C14, C15, C16, C17, C18, C19, C2, C20, C21, C22, C23, C24, C25, C26, C27, C28, C29, C3, C30, C31, C32, C33, C34, C35, C36, C37, C38, C39, C4, C40, C41, C42, C43, C44, C45, C46, C47, C48, C49, C5, C50, C51, C52, C53, C6, C7, C8, C9: 100nF, Capacitor_THT:C_Disc_D5.0mm_W2.5mm_P5.00mm, symbol p8x:CAP1
- removed LED3: GRN, LED_THT:LED_D5.0mm, symbol p8x:LED
- removed RP1: 1K, Resistor_THT:R_Axial_DIN0207_L6.3mm_D2.5mm_P10.16mm_Horizontal, symbol p8x:RES
- added U30, U31, U33, U39: 74HCT138, Package_DIP:DIP-16_W7.62mm, symbol p8x:74138
- added U32: 74HCT139, Package_DIP:DIP-16_W7.62mm, symbol p8x:74139
- added U34: 74HCT02, Package_DIP:DIP-14_W7.62mm, symbol p8x:7402
- added U35: 74HCT14, Package_DIP:DIP-14_W7.62mm, symbol p8x:HEX14
- added U36: 74HCT244, Package_DIP:DIP-20_W7.62mm, symbol p8x:74244
- added U37, U38: 74HCT08, Package_DIP:DIP-14_W7.62mm, symbol p8x:GATES14
- added U40, U53: 74HCT32, Package_DIP:DIP-14_W7.62mm, symbol p8x:GATES14
Connections:
- net GND: now also U30.4 (!G2A), U30.5 (!G2B), U30.8, U31.4 (!G2A), U31.5 (!G2B), U31.8, U32.8, U33.4 (!G2A), U33.5 (!G2B), U33.8, U34.11 (4A), U34.12 (4B), U34.5 (2A), U34.6 (2B), U34.7, U34.8 (3A), U34.9 (3B), U35.11 (5A), U35.13 (6A), U35.5 (3A), U35.7, U35.9 (4A), U36.10, U36.11 (A5), U36.13 (A6), U36.15 (A7), U36.17 (A8), U36.2 (A1), U36.4 (A2), U36.6 (A3), U36.8 (A4), U37.7, U38.10 (3B), U38.12 (4A), U38.13 (4B), U38.7, U38.9 (3A), U39.5 (!G2B), U39.8, U40.7, U53.10 (3B), U53.12 (4A), U53.13 (4B), U53.7, U53.9 (3A)
- net LDK: now also U38.6 (2Y)
- net RDK: now also U38.3 (1Y)
- net VCC: now also U30.16, U31.16, U32.16, U33.16, U33.6 (G1), U34.14, U35.14, U36.20, U37.14, U38.14, U39.16, U39.6 (G1), U40.14, U53.14
- new net -CNT0: U39.15 (Y0)
- new net -CNT1: U39.14 (Y1)
- new net -CNT2: U39.13 (Y2)
- new net -CNT3: U39.12 (Y3)
- new net -CNT4: U39.11 (Y4)
- new net -CNT5: U39.10 (Y5)
- new net -LDH: U30.14 (Y1), U37.13 (4B), U40.12 (4A), U40.4 (2A), U53.4 (2A)
- new net -LDH0: U32.12 (2Y0), U37.4 (2A)
- new net -LDH0E: U37.6 (2Y)
- new net -LDH1: U32.11 (2Y1)
- new net -LDH2: U32.10 (2Y2)
- new net -LDH3: U32.9 (2Y3)
- new net -LDH4: U40.11 (4Y)
- new net -LDH5: U53.6 (2Y)
- new net -LDHG: U32.15 (!G2), U40.6 (2Y)
- new net -LDL: U30.15 (Y0), U37.12 (4A), U40.1 (1A), U40.9 (3A), U53.1 (1A)
- new net -LDL0: U32.4 (1Y0), U37.1 (1A)
- new net -LDL0E: U37.3 (1Y)
- new net -LDL1: U32.5 (1Y1)
- new net -LDL2: U32.6 (1Y2)
- new net -LDL3: U32.7 (1Y3)
- new net -LDL4: U40.8 (3Y)
- new net -LDL5: U53.3 (1Y)
- new net -LDLG: U32.1 (!G1), U40.3 (1Y)
- new net -LDP: U37.11 (4Y), U38.4 (2A), U38.5 (2B)
- new net -POE: U37.8 (3Y), U38.1 (1A), U38.2 (1B)
- new net -POEH: U31.14 (Y1), U35.3 (2A), U37.10 (3B)
- new net -POEL: U31.15 (Y0), U37.9 (3A)
- new net -RES: U36.1 (!G1), U36.19 (!G2), U37.2 (1B), U37.5 (2B)
- new net -SEL0: U33.15 (Y0)
- new net -SEL1: U33.14 (Y1)
- new net -SEL2: U33.13 (Y2)
- new net -SEL3: U33.12 (Y3)
- new net -SEL4: U33.11 (Y4), U40.10 (3B), U40.13 (4B)
- new net -SEL5: U33.10 (Y5), U53.2 (1B), U53.5 (2B)
- new net CNTN: U34.1 (1Y), U39.4 (!G2A)
- new net D0: U36.18 (Y1)
- new net D1: U36.16 (Y2)
- new net D2: U36.14 (Y3)
- new net D3: U36.12 (Y4)
- new net D4: U36.9 (Y5)
- new net D5: U36.7 (Y6)
- new net D6: U36.5 (Y7)
- new net D7: U36.3 (Y8)
- new net DLD0: U30.1 (A)
- new net DLD1: U30.2 (B)
- new net DLD2: U30.3 (C)
- new net DLD3: U30.6 (G1)
- new net DOE0: U31.1 (A)
- new net DOE1: U31.2 (B)
- new net DOE2: U31.3 (C)
- new net DOE3: U31.6 (G1)
- new net PDEC: U34.3 (1B), U35.1 (1A)
- new net PINC: U34.2 (1A)
- new net POEHP: U35.4 (2Y)
- new net PSEL0: U32.14 (A2), U32.2 (A1), U33.1 (A), U39.1 (A)
- new net PSEL1: U32.13 (B2), U32.3 (B1), U33.2 (B), U39.2 (B)
- new net PSEL2: U33.3 (C), U39.3 (C), U40.2 (1B), U40.5 (2B)
- new net UDB: U35.2 (1Y)
- no-connect marks 0 -> 27
Other:
- moved on the sheet: LED4, LED5, R4, R5
