File: hardware/alu-card/kicad/p8x-alu-card-3.kicad_sch (KiCad schematic)
At the start: 9 parts, among them U19 74HCT08, U20 74HCT138, U21 74HCT138, U22 74HCT157, U23 74HCT244, U24 74HCT32, U25 74HCT00, U26 74HCT74, U27 74HCT260

Commit message: feat(sch): draw every P8X card schematic by function
Extend the functional-sheet grouping from the io-card to the control,
regbank, alu, memory, cf, ps2 and bustest cards. functional_sheets now
attaches unnamed glue gates, LEDs, resistors and connectors to the block
they share the most local nets with, so each block lists only its main
parts. A net with two or more pins on a sheet is now wired there even if
it continues elsewhere (its global name label rides on the wire), and
every wire is oriented by drawing side. The regbank gets one pointer per
sheet; the ps2 latches share a sheet with the AVR so the mailbox bus is
drawn. The bustest probe resistors use a straight-order RNISO8DSTR
drawing (the reversed B side forced every wire to cross and the sheet
fell back to labels). build_sch.sh now shows ELK fallbacks and clears old
numbered sheets before a build. All eight netlists match the boards,
ERC 0 errors; the boards change only in footprint link paths.

Co-Authored-By: Claude Opus 5.5 <noreply@anthropic.com>
Parts:
- removed U19: 74HCT08, Package_DIP:DIP-14_W7.62mm, symbol p8x:GATES14
- removed U20, U21: 74HCT138, Package_DIP:DIP-16_W7.62mm, symbol p8x:74138
- removed U22: 74HCT157, Package_DIP:DIP-16_W7.62mm, symbol p8x:74157
- removed U23: 74HCT244, Package_DIP:DIP-20_W7.62mm, symbol p8x:74244
- removed U24: 74HCT32, Package_DIP:DIP-14_W7.62mm, symbol p8x:GATES14
- removed U25: 74HCT00, Package_DIP:DIP-14_W7.62mm, symbol p8x:GATES14
- removed U26: 74HCT74, Package_DIP:DIP-14_W7.62mm, symbol p8x:7474
- removed U27: 74HCT260, Package_DIP:DIP-14_W7.62mm, symbol p8x:74260
- added U12, U13, U14, U15, U28, U30: 74HCT157, Package_DIP:DIP-16_W7.62mm, symbol p8x:74157
- added U16: 74HCT244, Package_DIP:DIP-20_W7.62mm, symbol p8x:74244
Connections:
- net -DOEALU: now also U16.1 (!G1), U16.19 (!G2)
- net D0: now also U16.18 (Y1)
- net D1: now also U16.16 (Y2)
- net D2: now also U16.14 (Y3)
- net D3: now also U16.12 (Y4)
- net D4: now also U16.9 (Y5)
- net D5: now also U16.7 (Y6)
- net D6: now also U16.5 (Y7)
- net D7: now also U16.3 (Y8)
- net FQC: now also U30.3 (B1)
- net GND: now also U12.15 (!G), U12.8, U13.15 (!G), U13.8, U14.15 (!G), U14.8, U15.15 (!G), U15.8, U16.10, U28.15 (!G), U28.8, U30.15 (!G), U30.8
- net R7: now also U15.12 (Y4), U16.17 (A8)
- net SH0: now also U12.1 (S), U13.1 (S), U28.1 (S)
- net SH1: now also U14.1 (S), U15.1 (S)
- net VCC: now also U12.16, U13.16, U14.16, U15.16, U16.20, U28.16, U30.16
- new net CIN: U30.2 (A1)
- new net F0: U12.2 (A1), U12.6 (B2), U28.2 (A1)
- new net F1: U12.10 (B3), U12.5 (A2)
- new net F2: U12.11 (A3), U12.13 (B4)
- new net F3: U12.14 (A4), U13.3 (B1)
- new net F4: U13.2 (A1), U13.6 (B2)
- new net F5: U13.10 (B3), U13.5 (A2)
- new net F6: U13.11 (A3), U13.13 (B4)
- new net F7: U13.14 (A4), U28.3 (B1)
- new net G0: U12.4 (Y1), U14.2 (A1)
- new net G1: U12.7 (Y2), U14.3 (B1), U14.5 (A2)
- new net G2: U12.9 (Y3), U14.11 (A3), U14.6 (B2)
- new net G3: U12.12 (Y4), U14.10 (B3), U14.14 (A4)
- new net G4: U13.4 (Y1), U14.13 (B4), U15.2 (A1)
- new net G5: U13.7 (Y2), U15.3 (B1), U15.5 (A2)
- new net G6: U13.9 (Y3), U15.11 (A3), U15.6 (B2)
- new net G7: U13.12 (Y4), U15.10 (B3), U15.14 (A4)
- new net R0: U14.4 (Y1), U16.2 (A1)
- new net R1: U14.7 (Y2), U16.4 (A2)
- new net R2: U14.9 (Y3), U16.6 (A3)
- new net R3: U14.12 (Y4), U16.8 (A4)
- new net R4: U15.4 (Y1), U16.11 (A5)
- new net R5: U15.7 (Y2), U16.13 (A6)
- new net R6: U15.9 (Y3), U16.15 (A7)
- new net SHCIN: U30.1 (S)
- new net SHIN: U12.3 (B1), U15.13 (B4), U30.4 (Y1)
- new net SHOUT: U28.4 (Y1)
