File: hardware/alu-card/kicad/p8x-alu-card-4.kicad_sch (KiCad schematic)
At the start: 8 parts, among them U28 74HCT157, U29 74HCT157, U30 74HCT157, U31 74HCT08, U32 74HCT157, U33 74HCT157, U34 74HCT86, U35 74HCT08

Commit message: feat(sch): draw every P8X card schematic by function
Extend the functional-sheet grouping from the io-card to the control,
regbank, alu, memory, cf, ps2 and bustest cards. functional_sheets now
attaches unnamed glue gates, LEDs, resistors and connectors to the block
they share the most local nets with, so each block lists only its main
parts. A net with two or more pins on a sheet is now wired there even if
it continues elsewhere (its global name label rides on the wire), and
every wire is oriented by drawing side. The regbank gets one pointer per
sheet; the ps2 latches share a sheet with the AVR so the mailbox bus is
drawn. The bustest probe resistors use a straight-order RNISO8DSTR
drawing (the reversed B side forced every wire to cross and the sheet
fell back to labels). build_sch.sh now shows ELK fallbacks and clears old
numbered sheets before a build. All eight netlists match the boards,
ERC 0 errors; the boards change only in footprint link paths.

Co-Authored-By: Claude Opus 5.5 <noreply@anthropic.com>
Parts:
- removed U28, U30, U32, U33: 74HCT157, Package_DIP:DIP-16_W7.62mm, symbol p8x:74157
- added LED4: GRN, LED_THT:LED_D5.0mm, symbol p8x:LED
- added LED5: YEL, LED_THT:LED_D5.0mm, symbol p8x:LED
- added R4, R5: 1K, Resistor_THT:R_Axial_DIN0207_L6.3mm_D2.5mm_P10.16mm_Horizontal, symbol p8x:RES
- added U17: FLAGS, Package_DIP:DIP-16_W7.62mm, symbol p8x:74175
- added U18, U27: 74HCT260, Package_DIP:DIP-14_W7.62mm, symbol p8x:74260
- added U19: 74HCT08, Package_DIP:DIP-14_W7.62mm, symbol p8x:GATES14
- added U22: 74HCT157, Package_DIP:DIP-16_W7.62mm, symbol p8x:74157
- added U23: 74HCT244, Package_DIP:DIP-20_W7.62mm, symbol p8x:74244
- added U24: 74HCT32, Package_DIP:DIP-14_W7.62mm, symbol p8x:GATES14
- added U25: 74HCT00, Package_DIP:DIP-14_W7.62mm, symbol p8x:GATES14
- added U26: 74HCT74, Package_DIP:DIP-14_W7.62mm, symbol p8x:7474
Connections:
- net -CCLR: now also U26.1 (!1CLR)
- net -CLRCb: now also U25.11 (4Y)
- net -RES: now also U17.1 (!CLR)
- net CFLGI: now also U25.6 (2Y)
- net CLKFC: now also U26.3 (1CLK)
- net CLKFZN: now also U17.9 (CLK)
- net FENZN: now also U24.3 (1Y)
- net FQC: now also U23.11 (A5), U23.2 (A1), U26.5 (1Q)
- net GND: now also U17.8, U18.10 (E2), U18.7, U18.9 (D2), U19.12 (4A), U19.13 (4B), U19.7, U22.15 (!G), U22.8, U23.10, U23.19 (!G2), U24.10 (3B), U24.12 (4A), U24.13 (4B), U24.7, U24.9 (3A), U25.7, U26.11 (2CLK), U26.12 (2D), U26.7, U27.10 (E2), U27.7, U27.9 (D2)
- net LDF: now also U24.1 (1A), U25.10 (3B), U25.9 (3A)
- net NC: now also U26.2 (1D)
- net SH0: now also U24.4 (2A)
- net SHANY: now also U24.6 (2Y)
- net VCC: now also R4.1, R5.1, U17.16, U18.14, U19.14, U22.16, U23.20, U24.14, U25.14, U26.10 (!2PRE), U26.13 (!2CLR), U26.14, U27.14
- net VSRC: now also U17.12 (D3)
- new net -DOEALU: U19.10 (3B), U19.9 (3A)
- new net -DOEFLG: U23.1 (!G1)
- new net -SETCb: U25.3 (1Y), U26.4 (!1PRE)
- new net ALUK: LED4.1 (K), U19.8 (3Y)
- new net CFLG: U25.4 (2A), U25.5 (2B)
- new net CLRC: U25.12 (4A), U25.13 (4B)
- new net D0: U23.18 (Y1), U27.1 (A1)
- new net D1: U23.16 (Y2), U27.2 (B1)
- new net D2: U23.14 (Y3), U27.11 (C1)
- new net D3: U23.12 (Y4), U27.12 (D1)
- new net D4: U27.13 (E1)
- new net D5: U27.3 (A2)
- new net D6: U27.4 (B2)
- new net D7: U22.6 (B2), U27.5 (C2)
- new net FC: U23.9 (Y5)
- new net FN: U23.5 (Y7)
- new net FQN: U17.7 (Q2), U23.15 (A7), U23.6 (A3)
- new net FQV: U17.10 (Q3), U23.17 (A8), U23.8 (A4)
- new net FQZ: U17.2 (Q1), U23.13 (A6), U23.4 (A2)
- new net FV: U23.3 (Y8)
- new net FZ: U23.7 (Y6)
- new net LDFK: LED5.1 (K), U25.8 (3Y)
- new net LDZN: U22.1 (S), U24.2 (1B)
- new net LEDAL: LED4.2 (A), R4.2
- new net LEDLF: LED5.2 (A), R5.2
- new net NSRC: U17.5 (D2), U22.7 (Y2)
- new net R0: U18.1 (A1)
- new net R1: U18.2 (B1)
- new net R2: U18.11 (C1)
- new net R3: U18.12 (D1)
- new net R4: U18.13 (E1)
- new net R5: U18.3 (A2)
- new net R6: U18.4 (B2)
- new net R7: U18.5 (C2), U22.5 (A2)
- new net SETC: U25.1 (1A), U25.2 (1B)
- new net SH1: U24.5 (2B)
- new net ZBH: U19.5 (2B), U27.6 (Y2)
- new net ZBL: U19.4 (2A), U27.8 (Y1)
- new net ZBUS: U19.6 (2Y), U22.3 (B1)
- new net ZFLG: U19.3 (1Y), U22.2 (A1)
- new net ZH: U18.6 (Y2), U19.2 (1B)
- new net ZL: U18.8 (Y1), U19.1 (1A)
- new net ZSRC: U17.4 (D1), U22.4 (Y1)
Other:
- moved on the sheet: U29, U31, U34, U35
