File: hardware/cf-card/kicad/p8x-cf-card-1.kicad_sch (KiCad schematic)
At the start: 9 parts, among them U1 74HCT245, U2 74HCT30, U3 74HCT138, U4 74HCT138, U5 74HCT14, U6 74HCT10, U7 74HCT10, U8 74HCT08, U9 74HCT374

Commit message: feat(sch): draw every P8X card schematic by function
Extend the functional-sheet grouping from the io-card to the control,
regbank, alu, memory, cf, ps2 and bustest cards. functional_sheets now
attaches unnamed glue gates, LEDs, resistors and connectors to the block
they share the most local nets with, so each block lists only its main
parts. A net with two or more pins on a sheet is now wired there even if
it continues elsewhere (its global name label rides on the wire), and
every wire is oriented by drawing side. The regbank gets one pointer per
sheet; the ps2 latches share a sheet with the AVR so the mailbox bus is
drawn. The bustest probe resistors use a straight-order RNISO8DSTR
drawing (the reversed B side forced every wire to cross and the sheet
fell back to labels). build_sch.sh now shows ELK fallbacks and clears old
numbered sheets before a build. All eight netlists match the boards,
ERC 0 errors; the boards change only in footprint link paths.

Co-Authored-By: Claude Opus 5.5 <noreply@anthropic.com>
Parts:
- removed U1: 74HCT245, Package_DIP:DIP-20_W7.62mm, symbol p8x:74245
- removed U9: 74HCT374, Package_DIP:DIP-20_W7.62mm, symbol p8x:74374
- added LED4, LED6: YEL, LED_THT:LED_D5.0mm, symbol p8x:LED
- added R4, R6: 1K, Resistor_THT:R_Axial_DIN0207_L6.3mm_D2.5mm_P10.16mm_Horizontal, symbol p8x:RES
- added U11: 74HCT10, Package_DIP:DIP-14_W7.62mm, symbol p8x:7410
Connections:
- net -CFOE1: now also LED6.1 (K)
- net -IOR1: now also U11.12 (1Y)
- net -IOW1: now also U11.6 (2Y)
- net ACTK: now also LED4.1 (K)
- net CLKB: now also U11.13 (1C), U11.5 (2C)
- net GND: now also U11.10 (3B), U11.11 (3C), U11.7, U11.9 (3A)
- net RDP: now also U11.2 (1B)
- net SELP1: now also U11.1 (1A), U11.3 (2A)
- net VCC: now also R4.1, R6.1, U11.14
- net WRP: now also U11.4 (2B)
- new net LEDAC: LED4.2 (A), R4.2
- new net LEDAC1: LED6.2 (A), R6.2
- no-connect marks 25 -> 18
Other:
- moved on the sheet: U2, U3, U4, U5, U6, U7, U8
