File: hardware/control-card/kicad/p8x-control-card-5.kicad_sch (KiCad schematic)
At the start: 34 parts

Commit message: feat(sch): draw every P8X card schematic by function
Extend the functional-sheet grouping from the io-card to the control,
regbank, alu, memory, cf, ps2 and bustest cards. functional_sheets now
attaches unnamed glue gates, LEDs, resistors and connectors to the block
they share the most local nets with, so each block lists only its main
parts. A net with two or more pins on a sheet is now wired there even if
it continues elsewhere (its global name label rides on the wire), and
every wire is oriented by drawing side. The regbank gets one pointer per
sheet; the ps2 latches share a sheet with the AVR so the mailbox bus is
drawn. The bustest probe resistors use a straight-order RNISO8DSTR
drawing (the reversed B side forced every wire to cross and the sheet
fell back to labels). build_sch.sh now shows ELK fallbacks and clears old
numbered sheets before a build. All eight netlists match the boards,
ERC 0 errors; the boards change only in footprint link paths.

Co-Authored-By: Claude Opus 5.5 <noreply@anthropic.com>
Parts:
- removed C1: 1uF, Capacitor_THT:C_Disc_D5.0mm_W2.5mm_P5.00mm, symbol p8x:CAP
- removed LED4: GRN, LED_THT:LED_D5.0mm, symbol p8x:LED
- removed LED5: RED, LED_THT:LED_D5.0mm, symbol p8x:LED
- removed R1, R2, R3: 10K, Resistor_THT:R_Axial_DIN0207_L6.3mm_D2.5mm_P10.16mm_Horizontal, symbol p8x:RES
- removed R4, R5: 1K, Resistor_THT:R_Axial_DIN0207_L6.3mm_D2.5mm_P10.16mm_Horizontal, symbol p8x:RES
- removed SWR, SWS, SWT: SPST, Button_Switch_THT:SW_PUSH_6mm, symbol p8x:SW2
- added J1: MABC96R, Connector_DIN:DIN41612_C_3x32_Male_Horizontal_THT, symbol p8x:DIN96C
Connections:
- net GND: now also J1.A31, J1.A32, J1.B11, J1.B13, J1.B15, J1.B17, J1.B19, J1.B21, J1.B23, J1.B25, J1.B3, J1.B31, J1.B32, J1.B5, J1.B7, J1.B9, J1.C31, J1.C32
- net VCC: now also J1.A1, J1.A2, J1.B1, J1.B2, J1.C1, J1.C2
- new net -RES: J1.A11
- new net ALUM: J1.C23
- new net ALUS0: J1.C19
- new net ALUS1: J1.C20
- new net ALUS2: J1.C21
- new net ALUS3: J1.C22
- new net BSEL: J1.B28
- new net CIN: J1.C24
- new net CLK: J1.A24
- new net CLKB: J1.A25
- new net CLRC: J1.B27
- new net D0: J1.A3
- new net D1: J1.A4
- new net D2: J1.A5
- new net D3: J1.A6
- new net D4: J1.A7
- new net D5: J1.A8
- new net D6: J1.A9
- new net D7: J1.A10
- new net DLD0: J1.A16
- new net DLD1: J1.A17
- new net DLD2: J1.A18
- new net DLD3: J1.A19
- new net DOE0: J1.A12
- new net DOE1: J1.A13
- new net DOE2: J1.A14
- new net DOE3: J1.A15
- new net FC: J1.A27
- new net FN: J1.A29
- new net FV: J1.A30
- new net FZ: J1.A28
- new net IRQ: J1.B29
- new net LDF: J1.A26
- new net LDZN: J1.C28
- new net PDEC: J1.A23
- new net PINC: J1.A22
- new net PSEL0: J1.A20
- new net PSEL1: J1.A21
- new net PSEL2: J1.C27
- new net SETC: J1.C30
- new net SH0: J1.C25
- new net SH1: J1.C26
- new net SHCIN: J1.C29
- no-connect marks 0 -> 29
Other:
- moved on the sheet: C10, C11, C12, C13, C14, C15, C16, C17, C18, C19, C2, C20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
