File: hardware/control-card/kicad/p8x-control-card-1.kicad_sch (KiCad schematic)
At the start: 9 parts, among them U1 74HCT161, U2 74HCT14, U3 74HCT74, U4 74HCT00, U5 74HCT08, U6 74HCT32, U7 74HCT377, U8 74HCT138, U9 74HCT151

Commit message: feat(sch): draw every P8X card schematic by function
Extend the functional-sheet grouping from the io-card to the control,
regbank, alu, memory, cf, ps2 and bustest cards. functional_sheets now
attaches unnamed glue gates, LEDs, resistors and connectors to the block
they share the most local nets with, so each block lists only its main
parts. A net with two or more pins on a sheet is now wired there even if
it continues elsewhere (its global name label rides on the wire), and
every wire is oriented by drawing side. The regbank gets one pointer per
sheet; the ps2 latches share a sheet with the AVR so the mailbox bus is
drawn. The bustest probe resistors use a straight-order RNISO8DSTR
drawing (the reversed B side forced every wire to cross and the sheet
fell back to labels). build_sch.sh now shows ELK fallbacks and clears old
numbered sheets before a build. All eight netlists match the boards,
ERC 0 errors; the boards change only in footprint link paths.

Co-Authored-By: Claude Opus 5.5 <noreply@anthropic.com>
Parts:
- removed U7: 74HCT377, Package_DIP:DIP-20_W7.62mm, symbol p8x:74377V2
- removed U8: 74HCT138, Package_DIP:DIP-16_W7.62mm, symbol p8x:74138
- removed U9: 74HCT151, Package_DIP:DIP-16_W7.62mm, symbol p8x:74151
- added C1: 1uF, Capacitor_THT:C_Disc_D5.0mm_W2.5mm_P5.00mm, symbol p8x:CAP
- added JP1: 1x4, Connector_PinHeader_2.54mm:PinHeader_1x04_P2.54mm_Vertical, symbol p8x:HDR4
- added LED4: GRN, LED_THT:LED_D5.0mm, symbol p8x:LED
- added LED5: RED, LED_THT:LED_D5.0mm, symbol p8x:LED
- added R1, R2, R3: 10K, Resistor_THT:R_Axial_DIN0207_L6.3mm_D2.5mm_P10.16mm_Horizontal, symbol p8x:RES
- added R4, R5: 1K, Resistor_THT:R_Axial_DIN0207_L6.3mm_D2.5mm_P10.16mm_Horizontal, symbol p8x:RES
- added SWR, SWS, SWT: SPST, Button_Switch_THT:SW_PUSH_6mm, symbol p8x:SW2
- added X1: 4MHZ, Oscillator:Oscillator_DIP-14, symbol p8x:OSC
Connections:
- net CLKRAW: now also JP1.2
- net DIVQA: now also JP1.3
- net DIVQB: now also JP1.4
- net GND: now also C1.2, SWR.1, SWS.1, SWT.1, X1.7
- net HALTK: now also LED5.1 (K)
- net OSCO: now also JP1.1, X1.8 (OUT)
- net RSTRAW: now also C1.1, R1.2, SWT.2
- net RUNLK: now also LED4.1 (K)
- net RUNSW: now also R3.2, SWR.2
- net STEPRAW: now also R2.2, SWS.2
- net VCC: now also R1.1, R2.1, R3.1, R4.1, R5.1, X1.14
- new net LEDHL: LED5.2 (A), R5.2
- new net LEDRN: LED4.2 (A), R4.2
- no-connect marks 17 -> 10
Other:
- moved on the sheet: U1, U2, U3, U4, U5, U6

Commit message: fix(control): clock select JP1 reaches /4 with one shunt
JP1 was a 1x4 header (1 = 4 MHz, 2 = CLKRAW, 3 = /2, 4 = /4), so 1 MHz
needed pins 2 and 4 joined -- a wire, not a shunt. It is now a 2x3 header
with CLKRAW on pins 2/4/6: a shunt on 1-2 = 4 MHz, 3-4 = 2 MHz, 5-6 = 1 MHz,
each row labelled on the silk. Board re-routed, check_card PASS, schematic
rebuilt (ERC 0). README no longer claims a /8 tap; the BOM lists 2x3
headers as pin headers.

Co-Authored-By: Claude Opus 5.5 <noreply@anthropic.com>
Parts:
- JP1: value 1x4 -> CLKSEL; footprint Connector_PinHeader_2.54mm:PinHeader_1x04_P2.54mm_Vertical -> Connector_PinHeader_2.54mm:PinHeader_2x03_P2.54mm_Vertical; symbol p8x:HDR4 -> p8x:JMP2X3
Connections:
- net CLKRAW: now also JP1.4, JP1.6
- net DIVQB: now also JP1.5; no longer JP1.4
Other:
- moved on the sheet: C1, LED4, LED5, R1, R2, R3, R4, R5, SWR, SWS, SWT, U1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
