File: hardware/control-card/kicad/p8x-control-card.kicad_pcb (KiCad board)
At the start: 4 copper layers, 280 x 140 mm, 58 parts, among them J1 MABC96R, U1 74HCT161, U10 28C64, U11 28C64, U12 28C64, U13 28C64, U14 74HCT374, U15 74HCT374, U16 74HCT374, U17 74HCT374, U18 74HCT161, U19 74HCT86, U2 74HCT14, U20 74HCT244, U21 74HCT74, U3 74HCT74, U4 74HCT00, U5 74HCT08, U6 74HCT32, U7 74HCT377, U8 74HCT138, U9 74HCT151, X1 4MHZ

Commit message: feat(boards): front-edge layout for switches, LEDs, connectors, jumpers
Apply the board layout rules to every P8X card (none built or
ordered): io-card switch, outward DB9s and LEDs on the front (right)
edge with the LED bars just inboard, jumpers and RTC on the bottom
edge; control-card buttons on the front edge and clock jumper on the
bottom edge; memory-card write-protect jumper on the top edge;
bustest Pico on the bottom edge with its USB end facing off the board,
probe header beside it. gen_kicad.py gains a PINNED table; the DSN
export routes to 0.21 mm so Freerouting's polygonised round pads no
longer produce 0.199 mm clearance misses. All four re-routed: PASS.

Co-Authored-By: Claude Opus 5.5 <noreply@anthropic.com>
Parts:
- moved SWR 111.2 mm to (264.8, 49.8)
- moved JP1 102.3 mm to (62.2, 130.0), turned to 90 degrees
- moved SWS 94.4 mm to (264.8, 65.8)
- moved SWT 79.9 mm to (264.8, 81.8)
Routing:
- net CLKRAW: track 112.8 -> 228.2 mm, vias 0 -> 1
- net RSTRAW: track 184.3 -> 291.7 mm
- net STEPRAW: track 164.0 -> 267.1 mm, vias 1 -> 2
- net RUNSW: track 91.0 -> 192.0 mm, vias 0 -> 2
- net P14B7: track 57.4 -> 85.6 mm, vias 2 -> 0
- net DIVQA: track 158.1 -> 134.0 mm, vias 2 -> 0
- net D4: track 247.6 -> 269.6 mm
- net OSCO: track 155.2 -> 173.5 mm, vias 2 -> 1
- net -RES: track 294.1 -> 276.1 mm, vias 1 -> 0
- net IRQ0: track 174.1 -> 156.7 mm, vias 0 -> 1
- net FCOND2: track 104.4 -> 120.0 mm, vias 2 -> 1
- net IRQ2: track 193.3 -> 178.1 mm
- net HALT: track 121.4 -> 135.6 mm, vias 2 -> 1
- net P14B4: track 63.8 -> 49.9 mm, vias 1 -> 0
- net BSEL: track 143.2 -> 130.0 mm, vias 2 -> 0
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
Commit message: feat(boards): silkscreen labels on every board
Apply the labelling rules to all nine boards: every reference printed
outside every part's courtyard (about 300 sat under their own chip),
the IC type or passive value beside it, function labels on every LED,
switch, jumper and cable connector in the same block as the reference,
and position labels (io DTE/NULL swap jumpers, input switch D0-D7 and
ON=0, bargraph end bits, control JP1 4M/OUT/2M/1M, backplane +5V/GND).

generators/silk_labels.py runs last in every board generator;
check_card.sh fails a board with a hidden reference or one under a
part. Build scripts gain REUSE_ROUTE=1 to re-import the existing
routing for a silkscreen-only change. The backplane mounting holes get
unique refs H1-H6 (six REF** let a routing re-import move one hole onto
another). gen_bom.py shares the chip-type table. All nine boards PASS.

Co-Authored-By: Claude Opus 5.5 <noreply@anthropic.com>
Other:
- board text added: "10K"
- board text added: "1K"
- board text added: "1M"
- board text added: "1uF"
- board text added: "2M"
- board text added: "4M"
- board text added: "4MHZ"
- board text added: "74HCT00"
- board text added: "74HCT08"
- board text added: "74HCT138"
- board text added: "74HCT14"
- board text added: "74HCT151"
- board text added: "74HCT161"
- board text added: "74HCT244"
- board text added: "74HCT32"
- board text added: "74HCT374"
- board text added: "74HCT377"
- board text added: "74HCT74"
- board text added: "74HCT86"
- board text added: "AT28C64"
- board text added: "OUT"

Commit message: fix(control): clock select JP1 reaches /4 with one shunt
JP1 was a 1x4 header (1 = 4 MHz, 2 = CLKRAW, 3 = /2, 4 = /4), so 1 MHz
needed pins 2 and 4 joined -- a wire, not a shunt. It is now a 2x3 header
with CLKRAW on pins 2/4/6: a shunt on 1-2 = 4 MHz, 3-4 = 2 MHz, 5-6 = 1 MHz,
each row labelled on the silk. Board re-routed, check_card PASS, schematic
rebuilt (ERC 0). README no longer claims a /8 tap; the BOM lists 2x3
headers as pin headers.

Co-Authored-By: Claude Opus 5.5 <noreply@anthropic.com>
Parts:
- JP1: value 1x4 -> CLKSEL; footprint PinHeader_1x04_P2.54mm_Vertical -> PinHeader_2x03_P2.54mm_Vertical
- moved JP1 1.80 mm to (63.5, 131.3)
Connections:
- JP1 pad 4: DIVQB -> CLKRAW
Routing:
- net P14B7: track 85.6 -> 55.0 mm
- net CLKRAW: track 228.2 -> 199.8 mm, vias 1 -> 0
- net PSEL2: track 83.3 -> 108.7 mm, vias 1 -> 2
- net IRQ5: track 168.2 -> 193.0 mm
- net DLD1: track 234.4 -> 257.5 mm
- net D1: track 254.2 -> 232.6 mm, vias 1 -> 3
- net P14B0: track 54.0 -> 72.1 mm, vias 0 -> 2
- net OSCO: track 173.5 -> 158.5 mm, vias 1 -> 2
- net HALT: track 135.6 -> 120.8 mm
- net CLK: track 283.6 -> 298.3 mm, vias 2 -> 1
- net HALTK: track 166.5 -> 180.5 mm
- net FCOND1: track 65.8 -> 79.1 mm, vias 1 -> 3
- net D3: track 247.7 -> 260.3 mm, vias 2 -> 1
- net IRQ3: track 178.3 -> 165.8 mm
- net P16B2: track 71.9 -> 83.6 mm, vias 0 -> 1
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Other:
- board text added: "CLOCK"
- board text removed: "CLKSEL"
- board text removed: "OUT"

Commit message: feat(boards): title block with cottageworker.com on every board
Board rule of 2026-10-26: cottageworker.com on the silkscreen of every
card, beside the board's name and revision. No board carried its name or
revision before. silk_labels.title_block() prints the name + revision
(from the card title; memory REV F, backplane REV A) with the site
beneath, front (right) edge first so it reads with the card installed.
All nine boards rebuilt with the routing reused (silk only); every
check_card PASS.

Co-Authored-By: Claude Opus 5.5 <noreply@anthropic.com>
Other:
- board text added: "P8X CONTROL/MICROCODE CARD REV B"
- board text added: "cottageworker.com"
