File: hardware/ps2-card/kicad/p8x-ps2-card-3.kicad_sch (KiCad schematic)
At the start: 4 parts, among them J1 MABC96R

Commit message: feat(sch): draw every P8X card schematic by function
Extend the functional-sheet grouping from the io-card to the control,
regbank, alu, memory, cf, ps2 and bustest cards. functional_sheets now
attaches unnamed glue gates, LEDs, resistors and connectors to the block
they share the most local nets with, so each block lists only its main
parts. A net with two or more pins on a sheet is now wired there even if
it continues elsewhere (its global name label rides on the wire), and
every wire is oriented by drawing side. The regbank gets one pointer per
sheet; the ps2 latches share a sheet with the AVR so the mailbox bus is
drawn. The bustest probe resistors use a straight-order RNISO8DSTR
drawing (the reversed B side forced every wire to cross and the sheet
fell back to labels). build_sch.sh now shows ELK fallbacks and clears old
numbered sheets before a build. All eight netlists match the boards,
ERC 0 errors; the boards change only in footprint link paths.

Co-Authored-By: Claude Opus 5.5 <noreply@anthropic.com>
Parts:
- removed JICSP: ICSP, Connector_PinHeader_2.54mm:PinHeader_2x03_P2.54mm_Vertical, symbol p8x:JMP2X3
- removed PS2A: PS2-KBD, symbol p8x:MINIDIN6
- removed PS2B: PS2-MOUSE, symbol p8x:MINIDIN6
- added C1, C10, C11, C12, C13, C2, C3, C4, C5, C6, C7, C8, C9: 100nF, Capacitor_THT:C_Disc_D5.0mm_W2.5mm_P5.00mm, symbol p8x:CAP1
- added LEDPWR: GRN, LED_THT:LED_D5.0mm, symbol p8x:LED
- added RPWR: 1K, Resistor_THT:R_Axial_DIN0207_L6.3mm_D2.5mm_P10.16mm_Horizontal, symbol p8x:RES
Connections:
- net GND: now also C1.2, C10.2, C11.2, C12.2, C13.2, C2.2, C3.2, C4.2, C5.2, C6.2, C7.2, C8.2, C9.2, LEDPWR.1 (K)
- net VCC: now also C1.1, C10.1, C11.1, C12.1, C13.1, C2.1, C3.1, C4.1, C5.1, C6.1, C7.1, C8.1, C9.1, RPWR.2
- new net LPWRA: LEDPWR.2 (A), RPWR.1
- no-connect marks 43 -> 39
Other:
- moved on the sheet: J1
