File: hardware/ps2-card/kicad/p8x-ps2-card.kicad_pcb (KiCad board)
At the start: 4 copper layers, 280 x 140 mm, 41 parts, among them J1 MABC96R, U1 74HCT30, U10 74HCT374, U11 74HCT244, U12 74HCT244, U13 PS/2 MCU, U2 74HCT138, U3 74HCT138, U4 WIN CMP, U5 74HCT138, U6 74HCT138, U7 74HCT374, U8 74HCT374, U9 74HCT374

Commit message: feat(boards): silkscreen labels on every board
Apply the labelling rules to all nine boards: every reference printed
outside every part's courtyard (about 300 sat under their own chip),
the IC type or passive value beside it, function labels on every LED,
switch, jumper and cable connector in the same block as the reference,
and position labels (io DTE/NULL swap jumpers, input switch D0-D7 and
ON=0, bargraph end bits, control JP1 4M/OUT/2M/1M, backplane +5V/GND).

generators/silk_labels.py runs last in every board generator;
check_card.sh fails a board with a hidden reference or one under a
part. Build scripts gain REUSE_ROUTE=1 to re-import the existing
routing for a silkscreen-only change. The backplane mounting holes get
unique refs H1-H6 (six REF** let a routing re-import move one hole onto
another). gen_bom.py shares the chip-type table. All nine boards PASS.

Co-Authored-By: Claude Opus 5.5 <noreply@anthropic.com>
Other:
- board text added: "10K"
- board text added: "1K"
- board text added: "470R"
- board text added: "4X10K"
- board text added: "74HCT138"
- board text added: "74HCT244"
- board text added: "74HCT30"
- board text added: "74HCT374"
- board text added: "74HCT688"
- board text added: "ATmega1284P"
- board text added: "ICSP"
- board text added: "KBD-RD"
- board text added: "KEY-AVAIL"
- board text added: "KEYBOARD"
- board text added: "MOUSE"
- board text added: "MSE-RD"
- board text added: "PWR"

Commit message: feat(boards): title block with cottageworker.com on every board
Board rule of 2026-10-26: cottageworker.com on the silkscreen of every
card, beside the board's name and revision. No board carried its name or
revision before. silk_labels.title_block() prints the name + revision
(from the card title; memory REV F, backplane REV A) with the site
beneath, front (right) edge first so it reads with the card installed.
All nine boards rebuilt with the routing reused (silk only); every
check_card PASS.

Co-Authored-By: Claude Opus 5.5 <noreply@anthropic.com>
Other:
- board text added: "P8X PS/2 CARD REV A"
- board text added: "cottageworker.com"
