File: hardware/bustest-card/kicad/p8x-bustest-card.kicad_pcb (KiCad board)
At the start: 4 copper layers, 280 x 140 mm, 41 parts, among them J1 MABC96R, J2 PROBE, U1 MCP23S17, U2 MCP23S17, U3 MCP23S17, U4 MCP23S17, U5 MCP23S17, U6 74HCT244, U7 74HCT244

Commit message: fix(bustest): join IRQ and SPARE12-19 to the bus connector
The schematic ERC flagged single-pin labels on the bus test card: U4.GPA6
was named -IRQ while the bus line on B29 is IRQ, and the card's used_bus
set excluded every SPARE* net, so both allocations floated on the routed
board. Name the pin IRQ and map U5 port B to SPARE12-19 (B4-B18, the
design doc's allocation; was SPARE12-17), add the SPARE field to the
firmware table, and re-route the board: DRC 0 unconnected, PASS;
schematic ERC 0 errors, 0 warnings.

Co-Authored-By: Claude Opus 5.5 <noreply@anthropic.com>
Connections:
- J1 pad b10: (no net) -> SPARE15
- J1 pad b12: (no net) -> SPARE16
- J1 pad b14: (no net) -> SPARE17
- J1 pad b16: (no net) -> SPARE18
- J1 pad b18: (no net) -> SPARE19
- J1 pad b29: (no net) -> IRQ
- J1 pad b4: (no net) -> SPARE12
- J1 pad b6: (no net) -> SPARE13
- J1 pad b8: (no net) -> SPARE14
- U4 pad 27: -IRQ -> IRQ
- U5 pad 7: (no net) -> SPARE18
- U5 pad 8: (no net) -> SPARE19
Routing:
- net IRQ: track 0.00 -> 171.6 mm
- net SPARE12: track 0.00 -> 86.5 mm, vias 0 -> 1
- net D0: track 182.4 -> 112.6 mm, vias 2 -> 0
- net SPARE13: track 0.00 -> 68.1 mm
- net A1: track 156.9 -> 90.6 mm
- net SPARE17: track 0.00 -> 65.4 mm, vias 0 -> 1
- net SPARE15: track 0.00 -> 64.8 mm, vias 0 -> 1
- net SPARE18: track 0.00 -> 64.3 mm, vias 0 -> 1
- net SPARE14: track 0.00 -> 64.2 mm, vias 0 -> 1
- net SPARE19: track 0.00 -> 64.0 mm, vias 0 -> 1
- net A3: track 149.5 -> 87.4 mm, vias 2 -> 0
- net SPARE16: track 0.00 -> 61.9 mm, vias 0 -> 1
- net A6: track 131.5 -> 86.4 mm, vias 3 -> 1
- net A4: track 114.4 -> 84.7 mm, vias 3 -> 0
- net A10: track 139.4 -> 114.9 mm
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
Commit message: fix(bustest,io): real Pico footprint and a CR2032 holder
The bus test card's Pico was a substituted 2x20 pin header (rows 2.54 mm
apart, odd/even numbering), so a Pico could not have been fitted; it is
now KiCad's Module:RaspberryPi_Pico_Common_THT (rows 17.78 mm, Pico pin
order) and all eight Pico ground pins are netted (only 3 and 33 were).
The io-card's CR2032 sat in a Keystone 3000 footprint, a 12 mm SMD
holder; it is now the through-hole Keystone 103 (20 mm) placed in the
free bottom-right corner beside J3. Both boards re-routed: DRC 0
unconnected, PASS. The remaining substitutions were audited; the open
ones (io-card RNISO8 SIP vs the DIP-16 rule, 8-segment DIP-16
bargraphs, the custom MiniDIN-6) are listed under VERIFY in BACKLOG.md.

Co-Authored-By: Claude Opus 5.5 <noreply@anthropic.com>
Parts:
- A1: footprint PinHeader_2x20_P2.54mm_Vertical -> RaspberryPi_Pico_Common_THT
- moved A1 181.1 mm to (34.7, 48.5)
- moved J2 45.8 mm to (114.0, 47.5)
- moved R6 45.8 mm to (61.3, 47.2)
- moved R7 45.8 mm to (78.6, 47.2)
- moved R8 45.8 mm to (96.0, 47.2)
Connections:
- A1 pad 13: (no net) -> GND
- A1 pad 18: (no net) -> GND
- A1 pad 23: (no net) -> GND
- A1 pad 28: (no net) -> GND
- A1 pad 38: (no net) -> GND
- A1 pad 8: (no net) -> GND
Routing:
- net P5V: track 88.8 -> 243.8 mm, vias 0 -> 3
- net ST7: track 42.7 -> 175.9 mm, vias 1 -> 0
- net P_MISO: track 194.8 -> 68.6 mm
- net ST6: track 46.6 -> 167.7 mm
- net ST5: track 46.4 -> 164.1 mm, vias 0 -> 2
- net ST4: track 46.4 -> 162.2 mm, vias 0 -> 1
- net ST3: track 51.8 -> 155.1 mm
- net P_SCK: track 152.5 -> 49.5 mm
- net ST2: track 53.1 -> 149.9 mm, vias 1 -> 0
- net ST1: track 54.6 -> 148.9 mm
- net P_SI: track 139.3 -> 59.5 mm
- net ST0: track 69.6 -> 142.8 mm
- net P_CS: track 134.3 -> 64.5 mm
- net DOE0: track 106.9 -> 170.7 mm, vias 1 -> 4
- net P_RST: track 134.9 -> 71.6 mm, vias 2 -> 0
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
Commit message: feat(boards): front-edge layout for switches, LEDs, connectors, jumpers
Apply the board layout rules to every P8X card (none built or
ordered): io-card switch, outward DB9s and LEDs on the front (right)
edge with the LED bars just inboard, jumpers and RTC on the bottom
edge; control-card buttons on the front edge and clock jumper on the
bottom edge; memory-card write-protect jumper on the top edge;
bustest Pico on the bottom edge with its USB end facing off the board,
probe header beside it. gen_kicad.py gains a PINNED table; the DSN
export routes to 0.21 mm so Freerouting's polygonised round pads no
longer produce 0.199 mm clearance misses. All four re-routed: PASS.

Co-Authored-By: Claude Opus 5.5 <noreply@anthropic.com>
Parts:
- moved A1 152.1 mm to (159.4, 135.5), turned to 180 degrees
- moved J2 86.0 mm to (93.6, 131.0), turned to 90 degrees
- moved R6 28.2 mm to (33.1, 47.2)
- moved R8 28.2 mm to (67.8, 47.2)
- moved R7 28.2 mm to (50.4, 47.2)
Routing:
- net PRJ0: track 84.8 -> 189.5 mm
- net ST7: track 175.9 -> 71.9 mm
- net SENSE5: track 249.7 -> 345.6 mm
- net ST5: track 164.1 -> 68.5 mm, vias 2 -> 0
- net ST6: track 167.7 -> 72.2 mm, vias 1 -> 0
- net PRJ1: track 89.3 -> 175.6 mm, vias 1 -> 2
- net ST4: track 162.2 -> 76.4 mm, vias 1 -> 0
- net PRJ3: track 94.5 -> 173.9 mm, vias 0 -> 2
- net PRJ5: track 100.9 -> 175.9 mm
- net PRJ4: track 100.6 -> 174.1 mm, vias 1 -> 0
- net ST2: track 149.9 -> 76.4 mm
- net PRJ6: track 106.0 -> 177.6 mm
- net P_SCK: track 49.5 -> 120.7 mm, vias 1 -> 0
- net PRJ7: track 107.9 -> 179.0 mm
- net DOE0: track 170.7 -> 100.5 mm, vias 4 -> 3
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
Commit message: feat(boards): silkscreen labels on every board
Apply the labelling rules to all nine boards: every reference printed
outside every part's courtyard (about 300 sat under their own chip),
the IC type or passive value beside it, function labels on every LED,
switch, jumper and cable connector in the same block as the reference,
and position labels (io DTE/NULL swap jumpers, input switch D0-D7 and
ON=0, bargraph end bits, control JP1 4M/OUT/2M/1M, backplane +5V/GND).

generators/silk_labels.py runs last in every board generator;
check_card.sh fails a board with a hidden reference or one under a
part. Build scripts gain REUSE_ROUTE=1 to re-import the existing
routing for a silkscreen-only change. The backplane mounting holes get
unique refs H1-H6 (six REF** let a routing re-import move one hole onto
another). gen_bom.py shares the chip-type table. All nine boards PASS.

Co-Authored-By: Claude Opus 5.5 <noreply@anthropic.com>
Other:
- board text added: "10K"
- board text added: "1K8"
- board text added: "3K3"
- board text added: "5V"
- board text added: "74HCT244"
- board text added: "8x1K"
- board text added: "8x330R"
- board text added: "ARM"
- board text added: "CKB"
- board text added: "CLK"
- board text added: "ERR"
- board text added: "LIS"
- board text added: "MCP23S17"
- board text added: "PICO (USB)"
- board text added: "PRB0"
- board text added: "PRB1"
- board text added: "PRB2"
- board text added: "PRB3"
- board text added: "PRB4"
- board text added: "PRB5"
- board text added: "PRB6"
- board text added: "PRB7"
- board text added: "RES"
- board text added: "Raspberry Pi Pico"
- board text added: "USB"
- board text removed: "GRN"
- board text removed: "RED"
- board text removed: "YEL"

Commit message: feat(boards): title block with cottageworker.com on every board
Board rule of 2026-10-26: cottageworker.com on the silkscreen of every
card, beside the board's name and revision. No board carried its name or
revision before. silk_labels.title_block() prints the name + revision
(from the card title; memory REV F, backplane REV A) with the site
beneath, front (right) edge first so it reads with the card installed.
All nine boards rebuilt with the routing reused (silk only); every
check_card PASS.

Co-Authored-By: Claude Opus 5.5 <noreply@anthropic.com>
Other:
- board text added: "P8X BUS TEST CARD V1.0"
- board text added: "cottageworker.com"
